File: Main_SMD_Controller.kicad_pcb (KiCad board)
At the start: 2 copper layers, 65 x 85 mm, 51 parts, among them J1 2.1-5.5 +12VDC, J10 Vsens, J11 Vin+, J12 Drain, J13 Gate, J14 Source, J2 Switch_Control, J3 +5V, J4 AnalogIO, J5 +12V, J7 VsensJMP, J8 Vin_-, J9 Conn_01x02, P1 Eoshi-chan_Silk, P2 Eoshi-chan_Silk, P3 Eoshi-chan_Silk, P4 Serial_QR, Q1 2N7002K, Q2 TK100E06N1, U1 NJM7805SDL1, U2 4066, U3 AD8226ARZ, U4 S-89713B-K8T2U

Commit message: Signed-off-by: EosinY <theodor338@gmail.com>
Parts:
- removed the P3 at (70.0, -44.0)
- removed Q2: TK100E06N1, Package_TO_SOT_THT:TO-220-3_Horizontal_TabDown
- C1: value 0.33u -> 0.47u
- C7: value 1000p -> 0.01u; footprint Capacitor_SMD:C_0603_1608Metric -> Capacitor_SMD:C_0402_1005Metric
- C8: footprint Capacitor_SMD:C_0603_1608Metric -> Capacitor_SMD:C_0402_1005Metric
- P1: moved to B.Cu
- P2: footprint Eoshi-chan_v2:Eoshi-chan-v2_15x15 -> Eoshi-chan_v2:Eoshi-chan-v2_10x10
- P3: renamed from P4; footprint JLCPCB_Serial:Serial_QR_8x8 -> JLCPCB_Serial:Serial_QR_5x5; moved to F.Cu
- U2: value 4066 -> TC74HC4066AF(F)
- moved P1 47.0 mm to (45.2, 39.7), turned to 180 degrees
- moved P3 11.4 mm to (35.1, 43.1), turned to 0 degrees
- moved P2 4.97 mm to (45.2, 45.1), turned to 0 degrees
- moved TH1 2.79 mm to (81.0, 62.2)
- moved U1 0.84 mm to (67.9, 106.0)
- renumbered J8 to J10, J9 to J11, J10 to J12, J11 to J13, J7 to J6, J12 to J7, J13 to J8, J14 to J9, R12 to R11, R11 to R12
Connections:
- net Net-(J2-Pad4) renamed /LOAD_ENABLE-G
- net Net-(J7-Pad2) renamed /Vmeas_IN
- net Net-(J9-Pad1) renamed /TH_1
- net Net-(J9-Pad2) renamed /TH_2
Routing:
- net /TH_2: track 6.35 -> 9.14 mm
- net /TH_1: track 6.35 -> 9.14 mm
- net /Vmeas: track 20.9 -> 21.6 mm
Other:
- board text added: "3 2 1"
- board text added: "80V, 5A, 100W"
- board text added: "Insert jumper pin"
- board text added: "Measure V from 3-2: IN+ 1-2: V SENS"
- board text added: "Thermister (to R11,12)"
- board text removed: "Thermister (to shunt resistor)"
