File: Main_SMD_Controller_2layer.kicad_pcb (KiCad board)
At the start: 4 copper layers, 65 x 85 mm, 59 parts, among them J1 2.1-5.5 +12VDC, J10 Vin_-, J11 Conn_01x02, J12 Vsens, J13 Vin+, J2 Switch_Control, J3 +5V, J4 AnalogIO, J5 +12V, J6 VsensJMP, J7 Drain, J8 Gate, J9 Source, P1 Eoshi-chan_Silk, P2 Eoshi-chan_Silk, P3 Serial_QR, Q1 2N7002K, U1 NJW4191M, U2 NJM7805SDL1, U3 TC74HC4066AP, U4 AD8226ARZ, U5 S-89713B-K8T2U

Commit message: fix pi controller
Parts:
- moved P2 1.70 mm to (45.0, 44.7)
- moved C8 1.27 mm to (53.1, 89.4), turned to -90 degrees
- moved D1 1.17 mm to (52.6, 45.7), turned to -90 degrees
- moved C6 1.08 mm to (54.0, 93.2), turned to 90 degrees
Connections:
- net /R+ renamed /MOS-
- net R- renamed Load-
Routing:
- net +12V: track 108.4 -> 114.3 mm, vias 1 -> 0
- net Load-: track 52.3 -> 54.6 mm
- net LOAD_ENABLE: track 59.8 -> 58.1 mm, vias 2 -> 0
- net /MOS-: track 16.5 -> 14.9 mm
- net Vconst_ENABLE: track 27.4 -> 28.6 mm, vias 1 -> 3
- net VEE: track 28.3 -> 28.1 mm, vias 4 -> 2
- net VCC: track 99.3 -> 99.2 mm, vias 3 -> 2
- net GND: vias 123 -> 125
Other:
- copper layers 4 -> 2
