File: Main_SMD_Controller_v2.kicad_sch (KiCad schematic)
At the start: 50 parts, among them J1 Vsens, J2 VsensJMP, J3 Vin+, J4 Drain, J7 Gate, J8 Source, J9 Vin_-, P1 Eoshi-chan_Silk, P2 Eoshi-chan_Silk, P3 Serial_QR, U10 TC74HC4066AP, U2 LT1167CN8, U3 TC74HC4066AP, U4 ADA4510-2ARZ, U6 ADA4522-1ARZ, U7 OP07, U9 AD633ANZ

Commit message: 電圧
Parts:
- added C10: C_Small, symbol Device:C_Small
- added R17: R, symbol Device:R
Connections:
- net BIAS: now also R4.2; no longer R16.2
- net GND: now also R16.2, R2.1, C10.2; no longer U4.3, U4.5
- net Vmeas: now also R17.1; no longer R1.1
- net Vmeas_IN: now also R1.2; no longer R4.2
- net at R16.1, U4.6: now also R17.2; no longer R1.2, R2.1
- net at R3.2, U4.2: now also U4.1; no longer R4.1
- new net: C10.1, R1.1, R2.2, U4.3
- new net: R3.1, R4.1, U4.5
Other:
- moved on the sheet: C1, C21, R11, R23, R7, U2, U6

Commit message: おおまか
Parts:
- removed C7, C8, C9: C_Small, symbol Device:C_Small
- removed R12: 200k, symbol Device:R
- removed R16, R17, R3, R4, R9: R, symbol Device:R
- removed R21: 10k, symbol Device:R
- removed unit 1 of U4
- added R1: 100k(1%), symbol Device:R
- added R11, R8: 20k(1), symbol Device:R
- added R13, R7: 10k(1), symbol Device:R
- added R2: 10k(1%), symbol Device:R
- added TP1: BIAS, symbol Connector:TestPoint_Probe
- added TP2: Pcalc, symbol Connector:TestPoint_Probe
- added TP3: Vmeas, symbol Connector:TestPoint_Probe
- added TP4: FeedBack, symbol Connector:TestPoint_Probe
- added TP5: Set, symbol Connector:TestPoint_Probe
- added TP6: Imeas, symbol Connector:TestPoint_Probe
- added TP7: R+, symbol Connector:TestPoint_Probe
- added TP8: R-, symbol Connector:TestPoint_Probe
- added unit 1 of U5
- C6: renamed from C21; value 0.01u -> 0.01u(FL)
- C7: renamed from C1; value 0.01u -> 0.01u(FL)
- C8: renamed from C10; value C_Small -> 0.001u
- R10: value R -> 39k(1)
- R12: renamed from R23; value 33k -> 33k(1)
- R16: renamed from R1; value R -> 510k(1)
- R17: renamed from R2; value R -> 10k(1)
- R3: renamed from R5; value R -> R(1)
- R4: renamed from R6; value R -> R(1)
- R5: renamed from R14; value R -> R(1)
- R6: renamed from R15; value R -> R(1)
- R9: renamed from R11; value 33k -> 10k(1)
- renumbered C2 to C1, C3 to C2, C4 to C3, C5 to C4, C6 to C5, J4 to J1, J7 to J2, J8 to J3, J2 to J4, J1 to J5, J3 to J6, J9 to J7, R7 to R14, R8 to R15, U10 to U1, U3 to U2, U7 to U3, U9 to U4, U4 to U5, U2 to U7
Connections:
- net ADC_Vref: now also R1.1
- net BIAS: now also U3.2 (-), R13.2, TP1.1
- net GND: now also U7.2, R2.2, TP8.1, U5.3; no longer R10.1, U3.3 (+)
- net Imeas: now also TP6.1
- net MOS_S: now also U7.3, TP7.1
- net Pcalc: now also TP2.1
- net VCC: now also U5.8 (VDD)
- net VEE: now also U5.4 (VSS)
- net Vmeas: now also R7.1, TP3.1
- net rt: now also TP5.1
- net yt: now also TP4.1
- net at U5.6: now also R10.1, R7.2, R8.1
- net Vin: now reaches C8.1, R16.1, R17.2
- net Vin: now also U5.5
- removed net Rs+: R10.2, U7.2, U7.3
- net Vmeas_IN: no longer names the net of J4.2 (Pin_2), R16.2
- new net: R1.2, R2.1, U3.3 (+)
- new net: R11.1, R8.2, U5.1
- new net: R10.2, R11.2, R13.1, U5.2
Other:
- note added: "0.1862V"
- note added: "0~52V"
- note added: "x2 (2.013)"
- moved on the sheet: C1, C2, C3, C4, C5, C6, C7, C8, H1, H2, H3, H4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

Commit message: sims
Parts:
- removed C1, C2, C3: 0.1u, Capacitor_SMD:C_0603_1608Metric, symbol Device:C_Small
- removed J5: Vsens, AM_Conn_ScrewTerminal:ScrewTerminal_01x01_PCB-20, symbol Connector:Screw_Terminal_01x01
- removed TP7: R+, symbol Connector:TestPoint_Probe
- removed TP8: R-, symbol Connector:TestPoint_Probe
- added C10, C11, C20, C21, C22, C23, C6, C7, C8, C9: 0.1u, Capacitor_SMD:C_0603_1608Metric, symbol Device:C_Small
- added J1: Sens, Connector_JST:JST_VH_B2P3-VH_1x02_P7.92mm_Vertical, symbol Connector_Generic:Conn_01x02
- added RV1, RV2, RV3, RV4: R_Trim, Potentiometer_THT:Potentiometer_Bourns_3296W_Vertical, symbol Device:R_Potentiometer_Trim
- C1: renamed from C8; footprint (none) -> Capacitor_SMD:C_0603_1608Metric
- C2: renamed from C6; footprint Capacitor_SMD:C_0402_1005Metric -> Capacitor_THT:C_Rect_L7.0mm_W2.5mm_P5.00mm
- C3: renamed from C7; footprint Capacitor_SMD:C_0402_1005Metric -> Capacitor_THT:C_Rect_L7.0mm_W2.5mm_P5.00mm
- C4, C5: Akizuki_code 116143 -> (none)
- D1: value GS1010FL -> 1N4007; footprint Diode_SMD:D_SOD-123 -> Diode_THT:D_DO-41_SOD81_P10.16mm_Horizontal
- R1: renamed from R10; footprint (none) -> Resistor_THT:R_Axial_DIN0207_L6.3mm_D2.5mm_P2.54mm_Vertical
- R10: renamed from R12; footprint (none) -> Resistor_THT:R_Axial_DIN0207_L6.3mm_D2.5mm_P2.54mm_Vertical
- R11: renamed from R14; footprint Resistor_SMD:R_0603_1608Metric -> Resistor_THT:R_Axial_DIN0207_L6.3mm_D2.5mm_P2.54mm_Vertical
- R12: renamed from R9; footprint (none) -> Resistor_THT:R_Axial_DIN0207_L6.3mm_D2.5mm_P2.54mm_Vertical
- R13: renamed from R3; footprint (none) -> Resistor_THT:R_Axial_DIN0207_L6.3mm_D2.5mm_P2.54mm_Vertical
- R14: renamed from R15; footprint Resistor_SMD:R_2512_6332Metric -> Resistor_THT:R_Bare_Metal_Element_L16.3mm_W4.8mm_P15.30mm
- R15: renamed from R4; footprint (none) -> Resistor_THT:R_Axial_DIN0207_L6.3mm_D2.5mm_P2.54mm_Vertical
- R16: renamed from R5; footprint (none) -> Resistor_THT:R_Axial_DIN0207_L6.3mm_D2.5mm_P2.54mm_Vertical
- R17: renamed from R6; footprint (none) -> Resistor_THT:R_Axial_DIN0207_L6.3mm_D2.5mm_P2.54mm_Vertical
- R2: renamed from R1; footprint (none) -> Resistor_THT:R_Axial_DIN0207_L6.3mm_D2.5mm_P2.54mm_Vertical
- R3: renamed from R11; footprint (none) -> Resistor_THT:R_Axial_DIN0207_L6.3mm_D2.5mm_P2.54mm_Vertical
- R4: renamed from R7; footprint (none) -> Resistor_THT:R_Axial_DIN0207_L6.3mm_D2.5mm_P2.54mm_Vertical
- R5: renamed from R2; footprint (none) -> Resistor_THT:R_Axial_DIN0207_L6.3mm_D2.5mm_P2.54mm_Vertical
- R6: renamed from R16; footprint (none) -> Resistor_THT:R_Axial_DIN0207_L6.3mm_D2.5mm_P2.54mm_Vertical
- R7: renamed from R13; footprint (none) -> Resistor_THT:R_Axial_DIN0207_L6.3mm_D2.5mm_P2.54mm_Vertical
- R8: footprint (none) -> Resistor_THT:R_Axial_DIN0207_L6.3mm_D2.5mm_P2.54mm_Vertical
- R9: renamed from R17; footprint (none) -> Resistor_THT:R_Axial_DIN0207_L6.3mm_D2.5mm_P2.54mm_Vertical
- TP1, TP4, TP5: footprint (none) -> TestPoint:TestPoint_Loop_D2.50mm_Drill1.0mm
- TP2: renamed from TP3; footprint (none) -> TestPoint:TestPoint_Loop_D2.50mm_Drill1.0mm
- TP3: renamed from TP2; footprint (none) -> TestPoint:TestPoint_Loop_D2.50mm_Drill1.0mm
- TP7: renamed from TP6; footprint (none) -> TestPoint:TestPoint_Loop_D2.50mm_Drill1.0mm
- U1: renamed from U3; footprint (none) -> Package_DIP:DIP-8_W7.62mm
- U2: renamed from U5; footprint Package_SO:SOP-8_3.9x4.9mm_P1.27mm -> Package_DIP:DIP-8_W7.62mm
- U4: renamed from U6; footprint Package_SO:SOP-8_3.9x4.9mm_P1.27mm -> Package_DIP:DIP-8_W7.62mm
- renumbered J4 to J2, J6 to J3, J1 to J4, J2 to J5, J3 to J6, U4 to U3, U2 to U5, U1 to U6
Connections:
- net +5V: now also C4.1, C5.1
- net GAIN_SEL2: now also RV1.1, RV1.2, RV2.1, RV2.2, RV3.1, RV3.2, RV4.1, RV4.2; no longer R13.2, R15.2, R16.2, R17.2
- net GND: now also C10.2, C11.2, C20.2, C21.2, C22.2, C23.2, C6.2, C7.2, C8.2, C9.2; no longer J5.2 (Pin_2), J7.1 (Pin_1), R14.2, R5.2, R9.1, RLY1.4 (NC), U2.3, U7.2
- net VCC: now also C10.1, C20.1, C22.1, C6.1, C8.1; no longer C4.1, C5.1
- net VEE: now also C11.1, C21.1, C23.1, C7.1, C9.1
- net Vin: now also R6.2; no longer R6.1
- net at R2.2, U1.3 (+): now also R5.2; no longer R5.1
- net at J2.1 (Pin_1): now also J1.1 (Pin_1)
- net at J2.2 (Pin_2): now also R6.1; no longer R6.2
- new net: R13.2, RV1.3
- new net: R15.2, RV2.3
- new net: R16.2, RV3.3
- new net: R17.2, RV4.3
- new net GNDA: J1.2 (Pin_2), J5.2 (Pin_2), J7.1 (Pin_1), R14.2, R5.1, R9.1, RLY1.4 (NC), U2.3, U7.2
Other:
- note removed: "4066のパスコン"
- note removed: "OPアンプのパスコン"
- moved on the sheet: C1, C2, C3, H1, H2, H3, H4, J2, P1, P2, P3, R1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

Commit message: もうだめだ  おしまいだ
Parts:
- removed TP3: Pcalc, TestPoint:TestPoint_Loop_D2.50mm_Drill1.0mm, symbol Connector:TestPoint_Probe
- removed U3: AD633ANZ, Package_DIP:DIP-8_W7.62mm, symbol AM_Opamp:AD633ANZ
- added C24: 0.1u, symbol Device:C_Small
- added C25, C26, C27, C28: 0.1u, Capacitor_SMD:C_0603_1608Metric, symbol Device:C_Small
- added J24: VsensJMP, Connector_PinHeader_2.54mm:PinHeader_1x03_P2.54mm_Vertical, symbol Connector_Generic:Conn_01x03
- added R28: 0, Resistor_THT:R_Axial_DIN0207_L6.3mm_D2.5mm_P2.54mm_Vertical, symbol Device:R
- added R29, R30: 10k(1), Resistor_THT:R_Axial_DIN0207_L6.3mm_D2.5mm_P2.54mm_Vertical, symbol Device:R
- added R31: 10k, Resistor_THT:R_Bare_Metal_Element_L16.3mm_W4.8mm_P15.30mm, symbol Device:R
- added R32: 10k, Resistor_THT:R_Axial_DIN0207_L6.3mm_D2.5mm_P2.54mm_Vertical, symbol Device:R
- added RV5: 50k, Potentiometer_THT:Potentiometer_Bourns_3296W_Vertical, symbol Device:R_Potentiometer_Trim
- added TP9: Vref, TestPoint:TestPoint_Loop_D2.50mm_Drill1.0mm, symbol Connector:TestPoint_Probe
- added U11: MCP1501-20E/CHY, Package_TO_SOT_SMD:SOT-23-6, symbol Reference_Voltage:MCP1501-20xCH
- added U12: KIA75S358F, Package_TO_SOT_SMD:SOT-23-5, symbol AM_Opamp:KIA75S358F
- added U3: CD4053B, symbol Analog_Switch:CD4053B
- added U9: NJU7098A, Package_TO_SOT_SMD:SOT-23-6, symbol AM_Opamp:NJU7098A
- C10, C2: now not fitted
- R10: value 33k(1) -> 0
- R11: value 100 -> 10k; footprint Resistor_THT:R_Axial_DIN0207_L6.3mm_D2.5mm_P2.54mm_Vertical -> Resistor_THT:R_Bare_Metal_Element_L16.3mm_W4.8mm_P15.30mm; Akizuki_code (none) -> 106668
- R12: value 10k(1) -> 10k
- TP1: value BIAS -> OFS
Connections:
- net Pcalc is gone; now on net Imeas: U6.4
- net +5V: now also C25.1, U11.4 (~{SHDN}), U11.6 (VDD)
- net AUX: now also U6.8; no longer U6.11
- net BIAS: no longer R7.2, TP1.1, U1.2 (-), U1.6, U7.5 (Ref)
- net GND: now also C25.2, C26.2, C27.2, C28.2, U11.2 (GND), U11.3 (GND), U11.5 (GND)
- net GNDA: now also R11.2, C24.2, R30.1, R31.2
- net Imeas: no longer U6.8
- net VCC: now also C11.1, C27.1, U9.6 (VDD); no longer C10.1
- net VEE: now also C26.1, C28.1, U9.2 (VEE); no longer C11.1
- net Vin: now also U9.3
- net Vmeas: now also J24.3 (Pin_3)
- net rt: now also R28.1; no longer U4.3
- net ut: now also C2.2, C3.2, R11.1, U4.6, U12.1; no longer J5.1 (Pin_1), R11.2
- net at R2.2, R5.2, U1.3 (+): now also C24.1
- net ADC_Vref: no longer names the net of R2.1
- net ADC_Vref: now also TP9.1, U11.1 (OUT)
- new net: C10.1, R28.2, U4.3
- new net: R31.1, R32.1, U12.3
- new net: R29.2, R30.2, U9.4
- new net: R32.2, RV5.3
- new net +12V: U12.5 (VCC)
- new net -12V: U12.2 (VEE)
- new net MOS_G: J5.1 (Pin_1), RV5.1, RV5.2, U12.4
- new net OFS: R7.2, TP1.1, U1.2 (-), U1.6, U7.5 (Ref)
- new net Vctrl: J24.1 (Pin_1)
- new net Vmeas_CR: R29.1, U9.1
Other:
- added sheet PIctrl (PIctrl.kicad_sch)
- sheet Interface ports: added none; removed ADC_Vref
- note added: "2.048V"
- note added: "V_{IN}=1/52*V_{SENS}"
- note added: "V_{MEAS}: 0~2V"
- note added: "V_{SENS}: 0~52V"
- note added: "f_{c}=160Hz"
- note added: "アナログPI制御 e(t)=[r(t)+V_{BIAS}]-[y(t)+V_{BIAS}]=r(t)-y(t) u(t)=P*e(t)+I*e(t) P=3.3 I=?"
- note added: "モード切替 A: CV B: CP C: CC D: その他(デジタルCR, デジタルCP) A,C: アナログCR"
- note removed: "0~52V"
- note removed: "x2 (2.013)"
- moved on the sheet: C20, C21, C22, C23, C3, C4, C5, C6, C7, C8, C9, D1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

Commit message: メインとPI制御の2分化
Parts:
- removed C11, C26, C5: 0.1u, Capacitor_SMD:C_0603_1608Metric, symbol Device:C_Small
- removed J24: VsensJMP, Connector_PinHeader_2.54mm:PinHeader_1x03_P2.54mm_Vertical, symbol Connector_Generic:Conn_01x03
- removed R29, R30: 10k(1), Resistor_THT:R_Axial_DIN0207_L6.3mm_D2.5mm_P2.54mm_Vertical, symbol Device:R
- removed U3: CD4053B, symbol Analog_Switch:CD4053B
- removed U6: TC74HC4066AP, Package_DIP:DIP-14_W7.62mm, symbol Analog_Switch:CD4066BE
- removed U9: NJU7098A, Package_TO_SOT_SMD:SOT-23-6, symbol AM_Opamp:NJU7098A
- C1: value 0.001u -> 1000p
- D1: value 1N4007 -> GS1010FL
Other:
- removed sheet PIctrl
- moved on the sheet: C1, C10, C2, C20, C21, C22, C23, C24, C25, C27, C28, C3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

Commit message: 半完成
Parts:
- removed C10, C22, C23, C27, C28: 0.1u, Capacitor_SMD:C_0603_1608Metric, symbol Device:C_Small
- removed C2, C3: 0.01u(FL), Capacitor_THT:C_Rect_L7.0mm_W2.5mm_P5.00mm, symbol Device:C_Small
- removed R10, R28: 0, Resistor_THT:R_Axial_DIN0207_L6.3mm_D2.5mm_P2.54mm_Vertical, symbol Device:R
- removed R11, R31: 10k, Resistor_THT:R_Bare_Metal_Element_L16.3mm_W4.8mm_P15.30mm, symbol Device:R
- removed R12, R32: 10k, Resistor_THT:R_Axial_DIN0207_L6.3mm_D2.5mm_P2.54mm_Vertical, symbol Device:R
- removed RV5: 50k, Potentiometer_THT:Potentiometer_Bourns_3296W_Vertical, symbol Device:R_Potentiometer_Trim
- removed TP4: FeedBack, TestPoint:TestPoint_Loop_D2.50mm_Drill1.0mm, symbol Connector:TestPoint_Probe
- removed TP5: Set, TestPoint:TestPoint_Loop_D2.50mm_Drill1.0mm, symbol Connector:TestPoint_Probe
- removed U1: OP07, Package_DIP:DIP-8_W7.62mm, symbol Amplifier_Operational:OP07
- removed U12: KIA75S358F, Package_TO_SOT_SMD:SOT-23-5, symbol AM_Opamp:KIA75S358F
- removed U4: ADA4522-1ARZ, Package_DIP:DIP-8_W7.62mm, symbol AM_Opamp:ADA4522-1ARZ
- added C26, C30, C31, C37, C38, C40, C41, C42, C43, C5: 0.1u, symbol Device:C_Small
- added C32, C33, C34, C35, C36, C39: 10u, symbol Device:C_Small
- added FB1, FB2, FB3, FB4: BLM21PG331SN, symbol Device:FerriteBead_Small
- added J23, J24: OP_PWR, AM_Conn_ScrewTerminal:EurostylePluggable_1x03_P5.08mm, symbol Connector_Generic:Conn_01x03
- added R47: 100, Resistor_THT:R_Axial_DIN0207_L6.3mm_D2.5mm_P2.54mm_Vertical, symbol Device:R
- added U1: NJU7098A, Package_TO_SOT_SMD:SOT-23-6, symbol AM_Opamp:NJU7098A
- added U6: XC6201P332MR-G, Package_TO_SOT_SMD:SOT-23-5, symbol AM_PowerIC_Linear:XC6201P332MR-G
- added U8: XC6201P502MR-G, Package_TO_SOT_SMD:SOT-23-5, symbol AM_PowerIC_Linear:XC6201P502MR-G
- added U9: XC6902N331MR-G, Package_TO_SOT_SMD:SOT-23-3, symbol AM_PowerIC_Linear:XC6902N331MR-G
- R2: value 100k(1%) -> 100k(0.1)
- R5: value 10k(1%) -> 10k(0.1)
Connections:
- net +12V: now also C36.1, C37.1, FB3.2, U8.1 (V_{IN})
- net +5V: now also C32.1, C5.1, FB1.2, U6.1 (V_{IN}); no longer C25.1, C4.1, U11.4 (~{SHDN}), U11.6 (VDD), U5.14 (V_{DD})
- net -12V: now also FB4.2
- net GND: now also C26.2, C30.2, C31.2, C32.2, C33.2, C34.2, C35.2, C36.2, C37.2, C38.2, C39.2, C40.2, C41.1, C42.2, C43.1, C5.2, J23.2 (Pin_2), J24.2 (Pin_2), U6.2 (GND), U8.2 (GND), U9.2 (GND)
- net OFS: now also R47.2, U1.1
- net at C24.1, R2.2, R5.2: now also U1.3
- net VCC renamed +3V3
- net +3V3: now also C25.1, U11.4 (~{SHDN}), U11.6 (VDD), C26.1, C33.1, U1.6 (VDD), U6.5 (V_{OUT})
- net VEE renamed -3V3
- net -3V3: now also C31.1, C35.1, U1.2 (VEE), U9.1 (-V_{OUT})
- new net: R47.1, U1.4
- new net: C40.1, FB1.1, J23.1 (Pin_1)
- new net: C43.2, FB4.1, J24.3 (Pin_3)
- new net: C41.2, FB2.1, J23.3 (Pin_3)
- new net: C42.1, FB3.1, J24.1 (Pin_1)
- new net +5VA: C38.1, C39.1, C4.1, U5.14 (V_{DD}), U8.5 (V_{OUT})
- new net -5V: C30.1, C34.1, FB2.2, U9.3 (-V_{IN})
- no-connect marks 2 -> 0
Other:
- added sheet PI (PI.kicad_sch)
- sheet Interface ports: added OFS, rt; removed 5V, AGND, AUX, AUX_SEL, BIAS, CC/CR, CP, CV, GND, Vcc, Vee, Vref
- note removed: "アナログPI制御 e(t)=[r(t)+V_{BIAS}]-[y(t)+V_{BIAS}]=r(t)-y(t) u(t)=P*e(t)+I*e(t) P=3.3 I=?"
- note removed: "モード切替 A: CV B: CP C: CC D: その他(デジタルCR, デジタルCP) A,C: アナログCR"
- moved on the sheet: C24, C25, C4, C6, C7, C8, C9, J6, J7, R13, R14, R15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

Commit message: aaaa
Parts:
- removed C31: 0.1u, symbol Device:C_Small
- removed C32, C34, C36: 10u, symbol Device:C_Small
- removed C4: 0.1u, Capacitor_SMD:C_0603_1608Metric, symbol Device:C_Small
- added C101, C102, C103: 47u, Capacitor_SMD:CP_Elec_6.3x5.9, symbol Device:C_Polarized_Small
- added C112, C126, C127: 0.1u, Capacitor_SMD:C_0603_1608Metric, symbol Device:C_Small
- added J104: PH-1X2SG, Connector_PinHeader_2.54mm:PinHeader_1x02_P2.54mm_Vertical, symbol Connector_Generic:Conn_01x02
- C104: renamed from C5; value 0.1u -> 1u; footprint (none) -> Capacitor_SMD:C_0603_1608Metric; Akizuki_code (none) -> 114526; Akizuki_code2 (none) -> 116994
- C105: renamed from C30; value 0.1u -> 1u; footprint (none) -> Capacitor_SMD:C_0603_1608Metric; Akizuki_code (none) -> 114526; Akizuki_code2 (none) -> 116994
- C106: renamed from C37; value 0.1u -> 1u; footprint (none) -> Capacitor_SMD:C_0603_1608Metric; Akizuki_code (none) -> 114526; Akizuki_code2 (none) -> 116994
- C107: renamed from C40; footprint (none) -> Capacitor_SMD:C_0603_1608Metric; Akizuki_code (none) -> 105728
- C108: renamed from C41; footprint (none) -> Capacitor_SMD:C_0603_1608Metric; Akizuki_code (none) -> 105728
- C109: renamed from C42; footprint (none) -> Capacitor_SMD:C_0603_1608Metric; Akizuki_code (none) -> 105728
- C110: renamed from C43; footprint (none) -> Capacitor_SMD:C_0603_1608Metric; Akizuki_code (none) -> 105728
- C111: renamed from C26; footprint (none) -> Capacitor_SMD:C_0603_1608Metric; Akizuki_code (none) -> 105728
- C113: renamed from C38; footprint (none) -> Capacitor_SMD:C_0603_1608Metric; Akizuki_code (none) -> 105728
- C114: renamed from C33; value 10u -> 4.7u; footprint (none) -> Capacitor_SMD:C_1210_3225Metric; Akizuki_code (none) -> 115634
- C115: renamed from C35; value 10u -> 4.7u; footprint (none) -> Capacitor_SMD:C_1210_3225Metric; Akizuki_code (none) -> 115634
- C116: renamed from C39; value 10u -> 4.7u; footprint (none) -> Capacitor_SMD:C_1210_3225Metric; Akizuki_code (none) -> 115634
- C117: renamed from C25; Akizuki_code (none) -> 105728
- C118: renamed from C20; Akizuki_code (none) -> 105728
- C119: renamed from C21; Akizuki_code (none) -> 105728
- C120: renamed from C24; value 0.1u -> NC; footprint (none) -> Capacitor_SMD:C_0603_1608Metric; now not fitted
- C121: renamed from C8; Akizuki_code (none) -> 105728
- C122: renamed from C9; Akizuki_code (none) -> 105728
- C123: renamed from C6; Akizuki_code (none) -> 105728
- C124: renamed from C7; Akizuki_code (none) -> 105728
- C125: renamed from C1; value 1000p -> NC; now not fitted
- FB101: renamed from FB1; footprint (none) -> Inductor_SMD:L_0805_2012Metric; Akizuki_code (none) -> 104053
- FB102: renamed from FB2; footprint (none) -> Inductor_SMD:L_0805_2012Metric; Akizuki_code (none) -> 104053
- FB103: renamed from FB3; footprint (none) -> Inductor_SMD:L_0805_2012Metric; Akizuki_code (none) -> 104053
- FB104: renamed from FB4; footprint (none) -> Inductor_SMD:L_0805_2012Metric; Akizuki_code (none) -> 104053
- J101: renamed from J23; value OP_PWR -> B3B-XH-A; Akizuki_code (none) -> 112248
- J102: renamed from J24; value OP_PWR -> B3B-XH-A; Akizuki_code (none) -> 112248
- J103: renamed from J5; value Gate -> B2B-XH-A
- J105: renamed from J1; value Sens -> B2B-XH-A; footprint Connector_JST:JST_VH_B2P3-VH_1x02_P7.92mm_Vertical -> Connector_JST:JST_XH_B2B-XH-A_1x02_P2.50mm_Vertical; Akizuki_code (none) -> 112247
- J106: renamed from J2; value VsensJMP -> PH-1X3SG
- J107: renamed from J4; value Drain -> PCB-20
- J108: renamed from J6; value Source -> PCB-20
- J109: renamed from J3; value Vin+ -> PCB-20
- J110: renamed from J7; value Vin_- -> PCB-20
- R101: renamed from R2; footprint Resistor_THT:R_Axial_DIN0207_L6.3mm_D2.5mm_P2.54mm_Vertical -> Resistor_SMD:R_0805_2012Metric
- R102: renamed from R5; footprint Resistor_THT:R_Axial_DIN0207_L6.3mm_D2.5mm_P2.54mm_Vertical -> Resistor_SMD:R_0805_2012Metric
- R103: renamed from R4; value 10k(1) -> 1k(0.1); footprint Resistor_THT:R_Axial_DIN0207_L6.3mm_D2.5mm_P2.54mm_Vertical -> Resistor_SMD:R_0805_2012Metric
- R104: renamed from R47; footprint Resistor_THT:R_Axial_DIN0207_L6.3mm_D2.5mm_P2.54mm_Vertical -> Resistor_SMD:R_0603_1608Metric
- R105: renamed from R8; value 20k(1) -> 10k(0.1); footprint Resistor_THT:R_Axial_DIN0207_L6.3mm_D2.5mm_P2.54mm_Vertical -> Resistor_SMD:R_0805_2012Metric
- R106: renamed from R1; value 39k(1) -> 2.2k(0.5); Marutsu_code (none) -> M0083-1404
- R107: renamed from R3; value 20k(1) -> 10k(0.1); footprint Resistor_THT:R_Axial_DIN0207_L6.3mm_D2.5mm_P2.54mm_Vertical -> Resistor_SMD:R_0805_2012Metric
- R108: renamed from R7; value 10k(1) -> 1k(0.1); footprint Resistor_THT:R_Axial_DIN0207_L6.3mm_D2.5mm_P2.54mm_Vertical -> Resistor_SMD:R_0805_2012Metric
- R109: renamed from R6; value 510k(1) -> 39k(0.5); Marutsu_code (none) -> M0223-1635
- R110: renamed from R9; value 10k(1) -> 1k(0.5); Marutsu_code (none) -> M0083-1389
- R111: renamed from R13; value R(1) -> R(0.5)
- R112: renamed from R15; value R(1) -> R(0.5)
- R113: renamed from R16; value R(1) -> R(0.5)
- R114: renamed from R17; value R(1) -> R(0.5)
- R115: renamed from R14; value 20m -> BR3FB10L0 (10m); Akizuki_code 106668 -> (none); Marutsu_code (none) -> M2807-4003
- TP101: renamed from TP9; value Vref -> RCTCTE; footprint TestPoint:TestPoint_Loop_D2.50mm_Drill1.0mm -> (none)
- TP102: renamed from TP2; value Vmeas -> RCTCTE; footprint TestPoint:TestPoint_Loop_D2.50mm_Drill1.0mm -> (none)
- TP103: renamed from TP1; value OFS -> RCTCTE; footprint TestPoint:TestPoint_Loop_D2.50mm_Drill1.0mm -> (none)
- TP104: renamed from TP7; value Imeas -> RCTCTE; footprint TestPoint:TestPoint_Loop_D2.50mm_Drill1.0mm -> (none)
- U105: renamed from U2; footprint Package_DIP:DIP-8_W7.62mm -> Package_SO:SOIC-8_3.9x4.9mm_P1.27mm; AkizukiCode 114063 -> (none); Akizuki_code2 (none) -> 114063
- U107: renamed from U5; value TC74HC4066AP -> TC4066BP
- renumbered D1 to D101, H1 to H101, H2 to H102, H3 to H103, H4 to H104, P1 to P101, P2 to P102, P3 to P103, RLY1 to RLY101, RV1 to RV101, RV2 to RV102, RV3 to RV103, RV4 to RV104, U6 to U101, U9 to U102, U8 to U103, U11 to U104, U1 to U106, U7 to U108
Connections:
- net +12V: now also C103.1
- net +3V3: now also U107.14 (V_{DD}), C126.1
- net +5V: now also C101.1
- net +5VA: no longer U107.14 (V_{DD})
- net -3V3: now also U107.7 (V_{SS}), C112.2, C127.1
- net -5V: now also C102.2
- net GND: now also C120.2, J103.2 (Pin_2), R102.1, C101.2, C102.1, C112.1, C126.2, C127.2, J104.2 (Pin_2); no longer C106.2, C113.2, C116.2, U107.7 (V_{SS})
- net GNDA: now also U105.5; no longer C120.2, J103.2 (Pin_2), R102.1, U105.3
- net OFS: now also J104.1 (Pin_1)
- net Vin: now also U105.3; no longer U105.5
- net LOAD_EN renamed RLY_LOUT
- new net: C103.2, C106.2, C113.2, C116.2
Other:
- sheet Interface ports: added RLY_LOUT; removed LOAD_EN
- note added: "MOSFET,IGBT: G BJT: B"
- note added: "MOSFET: D BJT,IGBT: C"
- note added: "MOSFET: S BJT,IGBT: E"
- note added: "R1"
- note added: "R2"
- note added: "R2/R1 == R4/R3"
- note added: "R3"
- note added: "R4"
- note added: "Rg"
- note added: "V_{IN}=1/40*V_{SENS}"
- note added: "V_{SENS}: 0~40V"
- note added: "V_{in1}"
- note added: "V_{in2}"
- note added: "V_{ref}"
- note added: "Vo := G(V_{in1}-V_{in2})+V_{ref} G := 1 + R4/R3 + 2*R2/Rg = 2.009"
- note added: "入力+"
- note added: "入力-"
- note removed: "V_{IN}=1/52*V_{SENS}"
- note removed: "V_{SENS}: 0~52V"
- moved on the sheet: C104, C105, C106, C111, C113, C114, C115, C116, C117, C118, C119, C121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

Commit message: kannsei
Parts:
- removed C103: 47u, Capacitor_SMD:CP_Elec_6.3x5.9, symbol Device:C_Polarized_Small
- removed C106: 1u, Capacitor_SMD:C_0603_1608Metric, symbol Device:C_Small
- removed C116: 4.7u, Capacitor_SMD:C_1210_3225Metric, symbol Device:C_Small
- removed C118, C119, C121: 0.1u, Capacitor_SMD:C_0603_1608Metric, symbol Device:C_Small
- removed P101: Eoshi-chan_Silk, Eoshi-chan:Eoshi-chan_logo_15x15, symbol Eoshi-chan:Eoshi-chan_Silk
- removed U103: XC6201P502MR-G, Package_TO_SOT_SMD:SOT-23-5, symbol AM_PowerIC_Linear:XC6201P502MR-G
- added C114, C123: 0.1u, Capacitor_SMD:C_0603_1608Metric, symbol Device:C_Small
- added R114: 0, Resistor_SMD:R_0805_2012Metric, symbol Device:R
- D101: footprint Diode_THT:D_DO-41_SOD81_P10.16mm_Horizontal -> Diode_SMD:D_SOD-123F
- J101: renamed from J102; value B3B-XH-A -> ETB43034G000Z
- J102: renamed from J101; value B3B-XH-A -> ETB43034G000Z
- TP101: renamed from TP102; footprint (none) -> AM_Conn_TP:RCTCE
- TP102: renamed from TP104; footprint (none) -> AM_Conn_TP:RCTCE
- TP103: renamed from TP101; footprint (none) -> AM_Conn_TP:RCTCE
- TP104: renamed from TP103; footprint (none) -> AM_Conn_TP:RCTCE
- renumbered C109 to C101, C110 to C102, C107 to C103, C108 to C104, C101 to C105, C102 to C106, C104 to C107, C105 to C108, C111 to C109, C112 to C110, C114 to C111, C115 to C112, C117 to C115, C126 to C116, C127 to C117, C125 to C118, C123 to C119, C124 to C120, C120 to C121, FB103 to FB101, FB104 to FB102, FB101 to FB103, FB102 to FB104, J105 to J103, J106 to J104, J107 to J105, J103 to J106, J108 to J107, J104 to J108, P102 to P101, P103 to P102, R103 to R101, R111 to R102, R112 to R103, R113 to R104, R114 to R105, R105 to R106, R106 to R107, R107 to R108, R108 to R109, R109 to R110, R110 to R111, R101 to R112, R102 to R113, R104 to R115, R115 to R116, U107 to U103, U105 to U104, U104 to U105, U108 to U106, U106 to U107
Connections:
- net +5VA is gone; now on net +3V3: C113.1
- net +3V3: now also C122.1
- net -3V3: now also C114.1, C123.1; no longer C122.1
- net GND: now also C113.2, C114.2, C123.2, R114.2; no longer C118.2
- net GNDA: now also C118.2, R114.1
- net +12V renamed VCC
- net -12V renamed VEE
Other:
- company: (none) -> EosinY
- title: (none) -> Analog Controller
- moved on the sheet: C101, C102, C103, C104, C105, C106, C107, C108, C109, C110, C111, C112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
