File: Main_SMD_Controller_v2.kicad_sch (KiCad schematic)
At the start: 80 parts, among them J101 ETB43034G000Z, J102 ETB43034G000Z, J103 PH-1X3SG, J104 B2B-XH-A, J105 B2P3-VH-3.3(LF)(SN), J106 PH-1X3SG, J107 PCB-20, J108 B2B-XH-A, J109 PCB-20, J110 PH-1X2SG, J111 PCB-20, J112 PCB-20, P101 Eoshi-chan_Silk, U101 XC6201P332MR-G, U102 XC6902N331MR-G, U103 TC4066BP, U104 ADA4510-2ARZ, U105 MCP1501-20E/CHY, U106 LT1167CN8, U107 NJU7098A

Commit message: できたかも
Parts:
- C101, C102, C103, C104, C111, C112, C115, C116, C117, C118, C119, C121, C122, C124, C125: Akizuki_code2 (none) -> 116143
- FB101, FB102: Akizuki_code 104053 -> 113369
- J101, J102: Akizuki_code 112248 -> 111600
- J104: Akizuki_code (none) -> 112247
- J105: value B2P3-VH-3.3(LF)(SN) -> B2P3-VH-3.3; Akizuki_code 112247 -> 115084
- R101, R109: Akizuki_code (none) -> 111796
- R106, R108, R114: Akizuki_code (none) -> 111797
- R112, R115: Sengoku_code (none) -> EEHD-57HU
- R113: Akizuki_code (none) -> 111798
- R116: value 100 -> 200; Akizuki_code (none) -> 106201
- TP101, TP102, TP103, TP104: Akizuki_code (none) -> 131773
- U101: Akizuki_code (none) -> 115649
- U102: Akizuki_code (none) -> 115651
- U103: Akizuki_code (none) -> 131725
- U104: Akizuki_code (none) -> 118321
- U105: Akizuki_code (none) -> 115203
- U106: value LT1167CN8 -> AD623ANZ; Akizuki_code (none) -> 112706
- U107: Akizuki_code (none) -> 114988
