File: _autosave-Main_SMD_Controller_v2.kicad_sch (KiCad schematic)
At the start: 50 parts, among them J1 Vsens, J2 VsensJMP, J3 Vin+, J4 Drain, J7 Gate, J8 Source, J9 Vin_-, P1 Eoshi-chan_Silk, P2 Eoshi-chan_Silk, P3 Serial_QR, U10 TC74HC4066AP, U2 LT1167CN8, U3 TC74HC4066AP, U4 ADA4510-2ARZ, U6 ADA4522-1ARZ, U7 OP07, U9 AD633ANZ

Commit message: 電圧なににしよ
Parts:
- removed R16, R3, R4: R, symbol Device:R
- removed U4: ADA4510-2ARZ, Package_SO:SOP-8_3.9x4.9mm_P1.27mm, symbol AM_Opamp:ADA4510-2ARZ
- added U4: ADA4522-1ARZ, Package_SO:SOP-8_3.9x4.9mm_P1.27mm, symbol AM_Opamp:ADA4522-1ARZ
Connections:
- net Vmeas: no longer R1.1
- net Vmeas_IN: now also R2.2
- net at R2.1: now also R1.1; no longer R1.2
