File: v2_interface.kicad_sch (KiCad schematic)
At the start: 47 parts, among them J10 Power, J11 Vref_Select, J12 AUX_Select, J8 DE9_Socket, J9 DB25_Socket, Q1 2N7002K, Q2 2N7002K, U10 MCP1501-20xCH, U8 MCP4922, U9 MCP3424x-xSL

Commit message: sims
Parts:
- removed J10: Power, AM_Conn_ScrewTerminal:TerminalReceptacle_1x04_P2.54mm, symbol Connector_Generic:Conn_01x04
- removed J8: DE9_Socket, AM_Conn_Dsub:Dsub-9P_2.77mm-2.84mm-8.08mmOffset, symbol Connector:DE9_Socket
- removed TP10: ~{LDAC}, symbol Connector:TestPoint_Probe
- removed TP11: SCK, symbol Connector:TestPoint_Probe
- removed TP12: ~{CS}, symbol Connector:TestPoint_Probe
- removed TP13: SDO, symbol Connector:TestPoint_Probe
- removed TP14: Reserved1, symbol Connector:TestPoint_Probe
- removed TP15: Reserved2, symbol Connector:TestPoint_Probe
- removed TP16: Reserved3, symbol Connector:TestPoint_Probe
- removed TP17: Reserved4, symbol Connector:TestPoint_Probe
- removed TP19: SCL, symbol Connector:TestPoint_Probe
- removed TP20: SDA, symbol Connector:TestPoint_Probe
- removed TP21: GAIN_0, symbol Connector:TestPoint_Probe
- removed TP22: GAIN_1, symbol Connector:TestPoint_Probe
- removed TP23: GAIN_2, symbol Connector:TestPoint_Probe
- removed TP24: GAIN_3, symbol Connector:TestPoint_Probe
- removed TP25: CV, symbol Connector:TestPoint_Probe
- removed TP26: CP, symbol Connector:TestPoint_Probe
- removed TP27: CC/CR, symbol Connector:TestPoint_Probe
- removed TP28: AUX_SEL, symbol Connector:TestPoint_Probe
- removed TP9: SDI, symbol Connector:TestPoint_Probe
- added C17, C18, C19: 0.1u, Capacitor_SMD:C_0603_1608Metric, symbol Device:C_Small
- added J11: AnalogIO, Connector_PinHeader_2.54mm:PinHeader_2x05_P2.54mm_Vertical, symbol Connector_Generic:Conn_02x05_Odd_Even
- added J14: I^{2}C_TP1, Connector_PinHeader_2.54mm:PinHeader_1x03_P2.54mm_Vertical, symbol Connector_Generic:Conn_01x03
- added J15: I^{2}C_TP2, Connector_PinHeader_2.54mm:PinHeader_1x03_P2.54mm_Vertical, symbol Connector_Generic:Conn_01x03
- added J16: SPI_TP1, Connector_PinHeader_2.54mm:PinHeader_1x04_P2.54mm_Vertical, symbol Connector_Generic:Conn_01x04
- added J17: SPI_TP2, Connector_PinHeader_2.54mm:PinHeader_1x04_P2.54mm_Vertical, symbol Connector_Generic:Conn_01x04
- added J18: 3P_TempSensor, Connector_PinSocket_2.54mm:PinSocket_1x03_P2.54mm_Vertical, symbol Connector_Generic:Conn_01x03
- added J19: TP, Connector_PinHeader_2.54mm:PinHeader_1x03_P2.54mm_Vertical, symbol Connector_Generic:Conn_01x03
- added J20: CS_TP, Connector_PinHeader_2.54mm:PinHeader_1x04_P2.54mm_Vertical, symbol Connector_Generic:Conn_01x04
- added J21: ModPower, Connector_PinHeader_2.00mm:PinHeader_2x02_P2.00mm_Vertical, symbol Connector_Generic:Conn_02x02_Odd_Even
- added J22: 5V_PWR, AM_Conn_ScrewTerminal:EurostylePluggable_1x02_P5.08mm, symbol Connector_Generic:Conn_01x02
- added J23: OP_PWR, AM_Conn_ScrewTerminal:EurostylePluggable_1x03_P5.08mm, symbol Connector_Generic:Conn_01x03
- added J8: GAIN_TP, Connector_PinHeader_2.54mm:PinHeader_1x04_P2.54mm_Vertical, symbol Connector_Generic:Conn_01x04
- added J9: MODE_TP, Connector_PinHeader_2.54mm:PinHeader_1x04_P2.54mm_Vertical, symbol Connector_Generic:Conn_01x04
- C12: renamed from C9; value C_Small -> 100p; footprint (none) -> Capacitor_SMD:C_0603_1608Metric
- C13: renamed from C12; value C_Small -> 1000p; footprint (none) -> Capacitor_SMD:C_0603_1608Metric
- C14: renamed from C10; value C_Small -> 100p; footprint (none) -> Capacitor_SMD:C_0603_1608Metric
- C15: renamed from C13; value C_Small -> 1000p; footprint (none) -> Capacitor_SMD:C_0603_1608Metric
- C16: renamed from C11; value C_Small -> 100p; footprint (none) -> Capacitor_SMD:C_0603_1608Metric
- R18: renamed from R19; value R -> 200; footprint (none) -> Resistor_SMD:R_0603_1608Metric
- R19: renamed from R20; value R -> 200; footprint (none) -> Resistor_SMD:R_0603_1608Metric
- R20: renamed from R24; footprint (none) -> Resistor_SMD:R_0603_1608Metric
- R21: renamed from R25; footprint (none) -> Resistor_SMD:R_0603_1608Metric
- R22: renamed from R21; value R -> 200; footprint (none) -> Resistor_SMD:R_0603_1608Metric
- R23: renamed from R22; value R -> 200; footprint (none) -> Resistor_SMD:R_0603_1608Metric
- R24: renamed from R23; value R -> 200; footprint (none) -> Resistor_SMD:R_0603_1608Metric
- R25: renamed from R26; footprint (none) -> Resistor_SMD:R_0603_1608Metric
- TP10: renamed from TP29; footprint (none) -> TestPoint:TestPoint_Loop_D2.50mm_Drill1.0mm
- TP9: renamed from TP18; footprint (none) -> TestPoint:TestPoint_Loop_D2.50mm_Drill1.0mm
- U10: renamed from U9; footprint Package_SO:SOIC-14_3.9x8.7mm_P1.27mm -> Package_DIP:DIP-14_W7.62mm
- U8: footprint (none) -> Package_DIP:DIP-14_W7.62mm
- renumbered J11 to J10, J9 to J13, Q2 to Q1, Q1 to Q2, R27 to R26, R18 to R27, U10 to U9
Connections:
- net TP4 is gone; now on net TP3: J13.25 (P25)
- net +5V: now also U10.9 (A0), C17.1, C18.1, C19.1, J18.1 (Pin_1), J21.1 (Pin_1), J21.3 (Pin_3), J22.1 (Pin_1)
- net AUX_Ext: now also J11.10 (Pin_10)
- net AUX_SEL: now also J9.4 (Pin_4)
- net BIAS: now also J11.6 (Pin_6)
- net CC/CR: now also J9.3 (Pin_3)
- net CP: now also J9.2 (Pin_2)
- net CV: now also J9.1 (Pin_1)
- net GAIN_0: now also J8.1 (Pin_1)
- net GAIN_1: now also J8.2 (Pin_2)
- net GAIN_2: now also J8.3 (Pin_3)
- net GAIN_3: now also J8.4 (Pin_4)
- net GND: now also J13.1, J13.13, J13.18 (P18), J13.21 (P21), J13.7, U10.10 (A1), U10.14 (CH4-), C17.2, C18.2, C19.2, J11.1 (Pin_1), J11.3 (Pin_3), J11.5 (Pin_5), J11.7 (Pin_7), J11.9 (Pin_9), J14.3 (Pin_3), J15.3 (Pin_3), J16.4 (Pin_4), J17.4 (Pin_4), J18.3 (Pin_3), J20.4 (Pin_4), J21.2 (Pin_2), J21.4 (Pin_4), J22.2 (Pin_2), J23.2 (Pin_2)
- net I^{2}C_SCL: now also J14.1 (Pin_1), J15.1 (Pin_1)
- net I^{2}C_SDA: now also J14.2 (Pin_2), J15.2 (Pin_2)
- net Imeas: now also J11.2 (Pin_2)
- net SPI_SCK: now also J16.1 (Pin_1), J17.1 (Pin_1)
- net SPI_SDI: now also J16.2 (Pin_2), J17.2 (Pin_2)
- net SPI_SDO: now also J16.3 (Pin_3), J17.3 (Pin_3)
- net TP1: now also J19.1 (Pin_1)
- net TP2: now also J13.12, J19.2 (Pin_2); no longer J13.24 (P24)
- net TP3: now also J19.3 (Pin_3); no longer J13.12
- net VCC: now also J23.1 (Pin_1)
- net VEE: now also J23.3 (Pin_3)
- net Vmeas: now also J11.4 (Pin_4)
- net Vref_Ext: now also J11.8 (Pin_8)
- net ~{DAC_CS}: now also J20.2 (Pin_2)
- net ~{DAC_LDAC}: now also J20.1 (Pin_1)
- net ATEMP: now reaches U10.13 (CH4+)
- net ATEMP: now also J18.2 (Pin_2)
- new net ~{CS}-Reserved1: J13.24 (P24), J20.3 (Pin_3)
Other:
- note added: "Address: 0b1101100 (0x6C)"
- moved on the sheet: C12, C13, C14, C15, C16, D2, J10, J12, Q1, Q2, R18, R19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

Commit message: もうだめだ  おしまいだ
Parts:
- removed TP9: ADC_Vref, TestPoint:TestPoint_Loop_D2.50mm_Drill1.0mm, symbol Connector:TestPoint_Probe
- removed U9: MCP1501-20xCH, Package_TO_SOT_SMD:SOT-23-6, symbol Reference_Voltage:MCP1501-20xCH
Connections:
- net ADC_Vref renamed ADC_ref

Commit message: メインとPI制御の2分化
Parts:
- removed J9: MODE_TP, Connector_PinHeader_2.54mm:PinHeader_1x04_P2.54mm_Vertical, symbol Connector_Generic:Conn_01x04
Connections:
- net AUX_SEL: no longer names the net of J13.5
- net CC/CR: no longer names the net of J13.17 (P17)
- net CP: no longer names the net of J13.4
- net CV: no longer names the net of J13.16 (P16)

Commit message: 半完成
Parts:
- removed C17, C18, C19: 0.1u, Capacitor_SMD:C_0603_1608Metric, symbol Device:C_Small
- removed J10: Vref_Select, Connector_PinHeader_2.54mm:PinHeader_1x03_P2.54mm_Vertical, symbol Connector_Generic:Conn_01x03
- removed J11: AnalogIO, Connector_PinHeader_2.54mm:PinHeader_2x05_P2.54mm_Vertical, symbol Connector_Generic:Conn_02x05_Odd_Even
- removed J12: AUX_Select, Connector_PinHeader_2.54mm:PinHeader_1x03_P2.54mm_Vertical, symbol Connector_Generic:Conn_01x03
- removed J13: DB25_Socket, AM_Conn_Dsub:Dsub-25P_2.77mm-2.84mm-8.08mmOffset, symbol Connector:DB25_Socket
- removed J14: I^{2}C_TP1, Connector_PinHeader_2.54mm:PinHeader_1x03_P2.54mm_Vertical, symbol Connector_Generic:Conn_01x03
- removed J15: I^{2}C_TP2, Connector_PinHeader_2.54mm:PinHeader_1x03_P2.54mm_Vertical, symbol Connector_Generic:Conn_01x03
- removed J16: SPI_TP1, Connector_PinHeader_2.54mm:PinHeader_1x04_P2.54mm_Vertical, symbol Connector_Generic:Conn_01x04
- removed J17: SPI_TP2, Connector_PinHeader_2.54mm:PinHeader_1x04_P2.54mm_Vertical, symbol Connector_Generic:Conn_01x04
- removed J18: 3P_TempSensor, Connector_PinSocket_2.54mm:PinSocket_1x03_P2.54mm_Vertical, symbol Connector_Generic:Conn_01x03
- removed J19: TP, Connector_PinHeader_2.54mm:PinHeader_1x03_P2.54mm_Vertical, symbol Connector_Generic:Conn_01x03
- removed J20: CS_TP, Connector_PinHeader_2.54mm:PinHeader_1x04_P2.54mm_Vertical, symbol Connector_Generic:Conn_01x04
- removed J21: ModPower, Connector_PinHeader_2.00mm:PinHeader_2x02_P2.00mm_Vertical, symbol Connector_Generic:Conn_02x02_Odd_Even
- removed J22: 5V_PWR, AM_Conn_ScrewTerminal:EurostylePluggable_1x02_P5.08mm, symbol Connector_Generic:Conn_01x02
- removed J23: OP_PWR, AM_Conn_ScrewTerminal:EurostylePluggable_1x03_P5.08mm, symbol Connector_Generic:Conn_01x03
- removed J8: GAIN_TP, Connector_PinHeader_2.54mm:PinHeader_1x04_P2.54mm_Vertical, symbol Connector_Generic:Conn_01x04
- removed U8: MCP4922, Package_DIP:DIP-14_W7.62mm, symbol Analog_DAC:MCP4922
- added C44, C45: 0.1u, Capacitor_SMD:C_0603_1608Metric, symbol Device:C_Small
- added J8: DE9_Socket, symbol Connector:DE9_Socket
- added J9: I2C_ex, symbol Connector_Generic:Conn_01x03
- added U3: MCP4725A0T-ECH, Package_TO_SOT_SMD:SOT-23-6, symbol Analog_DAC:MCP4725xxx-xCH
Connections:
- net ATEMP is gone; now on net GND: U10.13 (CH4+)
- net +5V: no longer U10.6 (V_{DD})
- net GAIN_0: now also J8.1
- net GAIN_1: now also J8.6
- net GAIN_2: now also J8.2
- net GAIN_3: now also J8.7
- net GND: now also C44.2, C45.2, J8.5, J8.8, J9.3 (Pin_3), U3.2 (VSS), U3.6 (A0)
- net I^{2}C_SCL: now also J8.4, J9.1 (Pin_1), U3.5 (SCL)
- net I^{2}C_SDA: now also J8.9, J9.2 (Pin_2), U3.4 (SDA)
- net ~{LOAD_G}: now also J8.3
- net BIAS renamed OFS
- net BIASmeas renamed OFSmeas
- new net +5VA: C44.1, C45.1, U10.6 (V_{DD}), U3.3 (VDD)
- new net rt: U3.1 (VOUT)
Other:
- note added: "Address: 0b1100000 (0x60)"
- moved on the sheet: C12, C13, C14, C15, C16, D2, Q1, Q2, R18, R19, R22, R23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

Commit message: aaaa
Parts:
- removed C44, C45: 0.1u, Capacitor_SMD:C_0603_1608Metric, symbol Device:C_Small
- removed J9: I2C_ex, symbol Connector_Generic:Conn_01x03
- removed Q2: 2N7002K, Package_TO_SOT_SMD:SOT-23, symbol Transistor_FET:2N7002K
- removed R27: 10k, Resistor_SMD:R_0603_1608Metric, symbol Device:R
- removed TP10: ~{LOAD_G}, TestPoint:TestPoint_Loop_D2.50mm_Drill1.0mm, symbol Connector:TestPoint_Probe
- added C301, C302, C303, C306: 0.1u, Capacitor_SMD:C_0603_1608Metric, symbol Device:C_Small
- added D301: OSBL1608C1A, LED_SMD:LED_0603_1608Metric, symbol Device:LED
- added D302: OSHR1608C1A, LED_SMD:LED_0603_1608Metric, symbol Device:LED
- added J302: PH-2x3SG, Connector_PinHeader_2.54mm:PinHeader_2x03_P2.54mm_Vertical, symbol Connector_Generic:Conn_02x03_Odd_Even
- added Q301, Q302, Q303: 2N7002K, Package_TO_SOT_SMD:SOT-23, symbol Transistor_FET:2N7002K
- added R301, R303, R307: 10k, Resistor_SMD:R_0603_1608Metric, symbol Device:R
- added R302, R304: 1k, Resistor_SMD:R_0603_1608Metric, symbol Device:R
- added R310, R311: 0, Resistor_SMD:R_0805_2012Metric, symbol Device:R
- added TP301: RCTCTE, symbol Connector:TestPoint_Probe
- added U301: SLG46826G, Package_SO:TSSOP-20_4.4x6.5mm_P0.65mm, symbol CPLD_Renesas:SLG46826G
- added U302: PCA9515AD, Package_SO:SOIC-8_3.9x4.9mm_P1.27mm, symbol AM_PLD:PCA9515AD
- added U305: MCP9701A-E_TO, digikey-footprints:TO-92-3, symbol dk_Temperature-Sensors-Analog-and-Digital-Output:MCP9701A-E_TO
- C304: renamed from C13; Akizuki_code (none) -> 102332; Sengoku_code (none) -> EEHD-6WFB
- C305: renamed from C15; Akizuki_code (none) -> 102332; Sengoku_code (none) -> EEHD-6WFB
- C307: renamed from C12; value 100p -> 1000p; Akizuki_code (none) -> 102332; Sengoku_code (none) -> EEHD-6WFB
- C308: renamed from C14; value 100p -> 1000p; Akizuki_code (none) -> 102332; Sengoku_code (none) -> EEHD-6WFB
- C309: renamed from C16; value 100p -> 1000p; Akizuki_code (none) -> 102332; Sengoku_code (none) -> EEHD-6WFB
- D303: renamed from D2; value OSR5PA5A33A-1MA -> OSYG1608; footprint LED_THT:LED_D5.0mm -> LED_SMD:LED_0603_1608Metric; Akizuki_code (none) -> 108275
- J301: renamed from J8; value DE9_Socket -> DMR-09PGG
- R305: renamed from R20; Akizuki_code (none) -> 106668
- R306: renamed from R21; Akizuki_code (none) -> 106668
- R308: renamed from R26; Akizuki_code (none) -> 106668
- R309: renamed from R25; value 10k -> 1k; Akizuki_code (none) -> 10668
- U304: renamed from U10; footprint Package_DIP:DIP-14_W7.62mm -> Package_SO:SOIC-14_3.9x8.7mm_P1.27mm
- renumbered Q1 to Q304, R18 to R312, R19 to R313, R22 to R314, R23 to R315, R24 to R316, U3 to U303
Connections:
- net GNDA is gone; now on net GND: U304.12 (CH3-)
- net +5V: now also C301.1, R302.1, R304.1, U302.8 (VCC); no longer U304.9 (A0)
- net +5VA: now also U304.9 (A0), C302.1, C303.1, C306.1, U301.20 (V_{DD}), U301.7 (V_{DD2}), U305.1 (VDD)
- net GAIN_0: now also U301.9 (IO7); no longer J301.1
- net GAIN_1: now also U301.8 (IO8); no longer J301.6
- net GAIN_2: now also U301.6 (IO9); no longer J301.2
- net GAIN_3: now also U301.5 (IO10); no longer J301.7
- net GND: now also C301.2, C302.2, C303.2, C306.2, R310.1, R311.1, U305.3 (GND); no longer J301.5, J301.8, Q304.2 (S), R308.1, U303.2 (VSS), U303.6 (A0), U304.10 (A1), U304.13 (CH4+), U304.5 (V_{SS})
- net Imeas+: now also U301.2 (IO13)
- net Vmeas+: now also U301.1 (IO14)
- net I^{2}C_SCL renamed SCL
- net SCL: now also J302.1 (Pin_1), J302.2 (Pin_2), U301.13 (SCL), U302.7 (SCL1); no longer J301.4
- net I^{2}C_SDA renamed SDA
- net SDA: now also J302.3 (Pin_3), J302.4 (Pin_4), U301.12 (SDA), U302.6 (SDA1); no longer J301.9
- net ~{LOAD_G}: no longer names the net of Q304.1 (G), R308.2
- net ~{LOAD_G}: now also Q303.1 (G), R307.2, TP301.1, U301.4 (IO11); no longer J301.3
- new net: Q301.1 (G), R301.2, U301.11 (IO6)
- new net: D302.1 (K), Q302.3 (D)
- new net: D302.2 (A), R304.2
- new net: D301.1 (K), Q301.3 (D)
- new net: D301.2 (A), R302.2
- new net: Q302.1 (G), R303.2, U301.14 (IO5)
- new net: J301.4, U302.2 (SCL0)
- new net: J301.9, U302.3 (SDA0)
- new net CAL_MODE: J301.3, U301.18 (IO1)
- new net EN: J301.8, U302.5 (EN)
- new net GAIN_0X: J301.1, U301.15 (IO4)
- new net GAIN_X0: J301.6, U301.16 (IO3)
- new net GNDD: J301.5, J302.5 (Pin_5), J302.6 (Pin_6), Q301.2 (S), Q302.2 (S), Q303.2 (S), Q304.2 (S), R301.1, R303.1, R307.1, R308.1, R310.2, R311.2, U301.10 (GND), U302.4 (GND), U303.2 (VSS), U303.6 (A0), U304.10 (A1), U304.5 (V_{SS})
- new net LOAD: J301.7, U301.19 (IO0)
- new net RLY_LOUT: Q303.3 (D)
- new net SAVE: J301.2, U301.17 (IO2)
- new net Temp: U301.3 (IO12), U304.13 (CH4+), U305.2 (VOUT)
Other:
- note added: "Load (YellowGreen)"
- note added: "No Fault (Blue)"
- note added: "Output Fault (Red)"
- note added: "外付け用兼ロジアナ用 使わないときはジャンパーをつけておく"
- moved on the sheet: C304, C305, C307, C308, C309, D303, J301, Q304, R305, R306, R308, R309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

Commit message: kannsei
Parts:
- removed J301: DMR-09PGG, symbol Connector:DE9_Socket
- removed R305: 10k, Resistor_SMD:R_0603_1608Metric, symbol Device:R
- removed U302: PCA9515AD, Package_SO:SOIC-8_3.9x4.9mm_P1.27mm, symbol AM_PLD:PCA9515AD
- added C302, C303, C304: 0.1u, Capacitor_SMD:C_0603_1608Metric, symbol Device:C_Small
- added J301: BH-14SG, Connector_IDC:IDC-Header_2x07_P2.54mm_Vertical, symbol Connector_Generic:Conn_01x14
- added Q303: BSS84, Package_TO_SOT_SMD:SOT-23, symbol Transistor_FET:BSS84
- added R301, R307, R308, R309, R310, R311, R312, R315, R317: 10k, Resistor_SMD:R_0603_1608Metric, symbol Device:R
- added U301: 74LCX541FT, Package_SO:TSSOP-20_4.4x6.5mm_P0.65mm, symbol 74xx:74LS541
- added U303: PCA9515AD, Package_SO:SOIC-8_3.9x4.9mm_P1.27mm, symbol AM_PLD:PCA9515AD
- TP301: footprint (none) -> AM_Conn_TP:RCTCE
- U305: renamed from U304; value MCP3424x-xSL -> MCP3424T-ESL
- renumbered C302 to C305, C303 to C306, C304 to C307, C305 to C308, C306 to C309, C307 to C310, C308 to C311, C309 to C312, Q303 to Q304, Q304 to Q305, R301 to R302, R302 to R303, R303 to R304, R304 to R305, R307 to R313, R308 to R314, R309 to R316, R310 to R318, R311 to R319, R312 to R320, R313 to R321, R314 to R322, R315 to R323, R316 to R324, U301 to U302, U303 to U304, U305 to U306
Connections:
- net +5V: no longer C301.1, R306.2
- net CAL_MODE: now also R306.2, U301.14 (Y4)
- net GAIN_0X: now also R317.2, U301.18 (Y0)
- net GAIN_X0: now also R315.2, U301.17 (Y1)
- net GND: no longer C301.2
- net GNDD: now also C301.2, R306.1, U305.9 (A0), C302.2, C303.2, C304.2, J301.11 (Pin_11), J301.14 (Pin_14), J301.3 (Pin_3), J301.7 (Pin_7), R307.1, R308.1, R310.1, R315.1, R317.1, U301.10 (GND), U301.11 (Y7), U301.12 (Y6), U301.13 (Y5), U301.7 (A5), U301.8 (A6), U301.9 (A7), U303.4 (GND)
- net LOAD: now also R308.2, U301.15 (Y3)
- net SAVE: now also R310.2, U301.16 (Y2)
- net SCL: now also R309.1, U303.7 (SCL1)
- net SDA: now also R311.1, U303.6 (SDA1); no longer R306.1
- net +5VA renamed +3V3
- net +3V3: now also C301.1, C302.1, C303.1, C304.1, Q303.2 (S), R301.2, R309.2, R311.2, R312.1, U301.20 (VCC), U303.8 (VCC); no longer U305.9 (A0)
- new net: J301.1 (Pin_1), U301.2 (A0)
- new net: J301.2 (Pin_2), U301.3 (A1)
- new net: J301.4 (Pin_4), U301.4 (A2)
- new net: J301.5 (Pin_5), U301.5 (A3)
- new net: J301.6 (Pin_6), U301.6 (A4)
- new net: J301.12 (Pin_12), U303.2 (SCL0)
- new net: J301.13 (Pin_13), U303.3 (SDA0)
- new net: Q303.3 (D), R307.2, U303.5 (EN)
- new net ~{EN}: J301.8 (Pin_8), Q303.1 (G), R301.1, R312.2, U301.1 (G1), U301.19 (G2)
- no-connect marks 0 -> 2
Other:
- note added: "Address: 0x60"
- note added: "Address: 0x6C"
- note removed: "Address: 0b1100000 (0x60)"
- note removed: "Address: 0b1101100 (0x6C)"
- note removed: "外付け用兼ロジアナ用 使わないときはジャンパーをつけておく"
- company: (none) -> EosinY
- title: (none) -> Analog Controller
- moved on the sheet: C305, C306, C307, C308, C309, C310, C311, C312, D301, D302, D303, Q301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
