File: v2_interface.kicad_sch (KiCad schematic)
At the start: 53 parts, among them J301 BH-14SG, J302 PH-2x3SG, Q301 2N7002K, Q302 2N7002K, Q303 BSS84, Q304 2N7002K, Q305 2N7002K, U301 74LCX541FT, U302 SLG46826G, U303 PCA9515AD, U304 MCP4725A0T-ECH, U305 MCP3424T-ESL, U306 MCP9701A-E_TO

Commit message: 念のため
Parts:
- U304: value MCP4725A0T-ECH -> MCP4726A0T-ECH
- U306: footprint digikey-footprints:TO-92-3 -> Package_TO_SOT_THT:TO-92_Inline
Connections:
- net GNDD: no longer U304.6 (A0)
- net Imeas+: now also U305.3 (CH2+); no longer U305.1 (CH1+)
- net Imeas-: now also U305.4 (CH2-); no longer U305.2 (CH1-)
- net OFSmeas: now also U305.13 (CH4+); no longer U305.11 (CH3+)
- net Temp: now also U305.11 (CH3+); no longer U305.13 (CH4+)
- net Vmeas+: now also U305.1 (CH1+); no longer U305.3 (CH2+)
- net Vmeas-: now also U305.2 (CH1-); no longer U305.4 (CH2-)
- new net ADC_Vref: U304.6 (V_{ref})
Changed lines of the file:
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@@
 	(wire
 		(pts
+			(xy 182.88 41.91) (xy 185.42 41.91)
+		)
+		(stroke
+			(width 0)
+			(type default)
+		)
+	)
+	(wire
+		(pts
 			(xy 62.23 22.86) (xy 66.04 22.86)
 		)
@@
 	(wire
 		(pts
+			(xy 210.82 101.6) (xy 214.63 101.6)
+		)
+		(stroke
+			(width 0)
+			(type default)
+		)
+	)
+	(wire
+		(pts
 			(xy 81.28 69.85) (xy 81.28 68.58)
 		)
@@
 	(wire
 		(pts
+			(xy 210.82 109.22) (xy 214.63 109.22)
+		)
+		(stroke
+			(width 0)
+			(type default)
+		)
+	)
+	(wire
+		(pts
 			(xy 139.7 31.75) (xy 139.7 44.45)
 		)
@@
 	(wire
 		(pts
-			(xy 210.82 106.68) (xy 214.63 106.68)
-		)
-		(stroke
-			(width 0)
-			(type default)
-		)
-	)
-	(wire
-		(pts
 			(xy 190.5 132.08) (xy 190.5 142.24)
 		)
@@
 	(wire
 		(pts
-			(xy 41.91 41.91) (xy 62.23 41.91)
+			(xy 210.82 99.06) (xy 214.63 99.06)
 		)
 		(stroke
@@
 	(wire
 		(pts
-			(xy 49.53 57.15) (xy 49.53 100.33)
+			(xy 41.91 41.91) (xy 62.23 41.91)
 		)
 		(stroke
@@
 	(wire
 		(pts
-			(xy 55.88 185.42) (xy 54.61 185.42)
+			(xy 49.53 57.15) (xy 49.53 100.33)
 		)
 		(stroke
@@
 	(wire
 		(pts
-			(xy 120.65 185.42) (xy 119.38 185.42)
+			(xy 55.88 185.42) (xy 54.61 185.42)
 		)
 		(stroke
@@
 	(wire
 		(pts
-			(xy 256.54 59.69) (xy 252.73 59.69)
+			(xy 120.65 185.42) (xy 119.38 185.42)
 		)
 		(stroke
@@
 	(wire
 		(pts
-			(xy 210.82 99.06) (xy 214.63 99.06)
+			(xy 256.54 59.69) (xy 252.73 59.69)
 		)
 		(stroke
@@
 	(wire
 		(pts
-			(xy 210.82 109.22) (xy 214.63 109.22)
-		)
-		(stroke
-			(width 0)
-			(type default)
-		)
-	)
-	(wire
-		(pts
 			(xy 30.48 64.77) (xy 33.02 64.77)
 		)
@@
 	(wire
 		(pts
-			(xy 210.82 101.6) (xy 214.63 101.6)
-		)
-		(stroke
-			(width 0)
-			(type default)
-		)
-	)
-	(wire
-		(pts
 			(xy 119.38 133.35) (xy 121.92 133.35)
 		)
@@
 	(wire
 		(pts
-			(xy 184.15 41.91) (xy 184.15 46.99)
-		)
-		(stroke
-			(width 0)
-			(type default)
-		)
-	)
-	(wire
-		(pts
 			(xy 30.48 34.29) (xy 62.23 34.29)
 		)
@@
 	(wire
 		(pts
-			(xy 185.42 41.91) (xy 184.15 41.91)
-		)
-		(stroke
-			(width 0)
-			(type default)
-		)
-	)
-	(wire
-		(pts
 			(xy 97.79 113.03) (xy 97.79 111.76)
 		)
@@
 	(wire
 		(pts
+			(xy 210.82 106.68) (xy 214.63 106.68)
+		)
+		(stroke
+			(width 0)
+			(type default)
+		)
+	)
+	(wire
+		(pts
 			(xy 95.25 185.42) (xy 96.52 185.42)
 		)
@@
 		)
 	)
+	(label "OFSmeas"
+		(at 214.63 121.92 0)
+		(effects
+			(font
+				(size 1.27 1.27)
+			)
+			(justify left bottom)
+		)
+	)
 	(label "SDA"
 		(at 177.8 104.14 180)
@@
 		)
 	)
+	(label "Vmeas+"
+		(at 214.63 99.06 0)
+		(effects
+			(font
+				(size 1.27 1.27)
+			)
+			(justify left bottom)
+		)
+	)
 	(label "SAVE"
 		(at 147.32 36.83 0)
@@
 		)
 	)
+	(label "Temp"
+		(at 214.63 114.3 0)
+		(effects
+			(font
+				(size 1.27 1.27)
+			)
+			(justify left bottom)
+		)
+	)
 	(label "CAL_MODE"
 		(at 147.32 41.91 0)
@@
 		)
 	)
+	(label "Imeas-"
+		(at 214.63 109.22 0)
+		(effects
+			(font
+				(size 1.27 1.27)
+			)
+			(justify left bottom)
+		)
+	)
 	(label "SCL"
 		(at 182.88 36.83 180)
@@
 		)
 	)
-	(label "Imeas"
-		(at 271.78 95.25 0)
+	(label "Imeas+"
+		(at 214.63 106.68 0)
 		(effects
 			(font
@@
 		)
 	)
-	(label "SCL"
-		(at 69.85 123.19 180)
+	(label "Imeas"
+		(at 271.78 95.25 0)
 		(effects
 			(font
 				(size 1.27 1.27)
 			)
-			(justify right bottom)
+			(justify left bottom)
 		)
 	)
 	(label "SCL"
-		(at 157.48 78.74 0)
+		(at 69.85 123.19 180)
 		(effects
 			(font
 				(size 1.27 1.27)
 			)
-			(justify left bottom)
+			(justify right bottom)
 		)
 	)
-	(label "Imeas-"
-		(at 214.63 101.6 0)
+	(label "SCL"
+		(at 157.48 78.74 0)
 		(effects
 			(font
@@
 		)
 	)
-	(label "Vmeas+"
-		(at 214.63 106.68 0)
-		(effects
-			(font
-				(size 1.27 1.27)
-			)
-			(justify left bottom)
-		)
-	)
-	(label "OFSmeas"
-		(at 214.63 114.3 0)
-		(effects
-			(font
-				(size 1.27 1.27)
-			)
-			(justify left bottom)
-		)
-	)
 	(label "Temp"
 		(at 95.25 135.89 0)
@@
 		)
 	)
+	(label "Vmeas-"
+		(at 214.63 101.6 0)
+		(effects
+			(font
+				(size 1.27 1.27)
+			)
+			(justify left bottom)
+		)
+	)
 	(label "OFS"
 		(at 271.78 137.16 0)
@@
 		)
 	)
-	(label "Imeas+"
-		(at 214.63 99.06 0)
-		(effects
-			(font
-				(size 1.27 1.27)
-			)
-			(justify left bottom)
-		)
-	)
 	(label "Imeas-"
 		(at 234.95 99.06 180)
@@
 		)
 	)
-	(label "Vmeas-"
-		(at 214.63 109.22 0)
-		(effects
-			(font
-				(size 1.27 1.27)
-			)
-			(justify left bottom)
-		)
-	)
 	(label "Temp"
 		(at 243.84 71.12 180)
@@
 		)
 	)
-	(label "Temp"
-		(at 214.63 121.92 0)
-		(effects
-			(font
-				(size 1.27 1.27)
-			)
-			(justify left bottom)
-		)
-	)
 	(label "LOAD"
 		(at 147.32 39.37 0)
@@
 		)
 	)
+	(hierarchical_label "ADC_Vref"
+		(shape input)
+		(at 182.88 41.91 180)
+		(effects
+			(font
+				(size 1.27 1.27)
+			)
+			(justify right)
+		)
+	)
 	(hierarchical_label "Imeas"
 		(shape input)
@@
 	)
 	(symbol
-		(lib_id "power:GNDD")
-		(at 184.15 46.99 0)
-		(unit 1)
-		(body_style 1)
-		(exclude_from_sim no)
-		(in_bom yes)
-		(on_board yes)
-		(in_pos_files yes)
-		(dnp no)
-		(fields_autoplaced yes)
-		(property "Reference" "#PWR0328"
-			(at 184.15 53.34 0)
-			(hide yes)
-			(show_name no)
-			(do_not_autoplace no)
-			(effects
-				(font
-					(size 1.27 1.27)
-				)
-			)
-		)
-		(property "Value" "GNDD"
-			(at 184.15 50.8 0)
-			(show_name no)
-			(do_not_autoplace no)
-			(effects
-				(font
-					(size 1.27 1.27)
-				)
-			)
-		)
-		(property "Footprint" ""
-			(at 184.15 46.99 0)
-			(hide yes)
-			(show_name no)
-			(do_not_autoplace no)
-			(effects
-				(font
-					(size 1.27 1.27)
-				)
-			)
-		)
-		(property "Datasheet" ""
-			(at 184.15 46.99 0)
-			(hide yes)
-			(show_name no)
-			(do_not_autoplace no)
-			(effects
-				(font
-					(size 1.27 1.27)
-				)
-			)
-		)
-		(property "Description" "Power symbol creates a global label with name \"GNDD\" , digital ground"
-			(at 184.15 46.99 0)
-			(hide yes)
-			(show_name no)
-			(do_not_autoplace no)
-			(effects
-				(font
-					(size 1.27 1.27)
-				)
-			)
-		)
-		(pin "1"
-		)
-		(instances
-			(project "Main_SMD_Controller_v2"
-				(path "/ad678d38-2bf7-47ec-94cd-212edb6f07b2/e2de0e16-a9d6-47f1-91b9-10aa4d2542d2"
-					(reference "#PWR0328")
-					(unit 1)
-				)
-			)
-		)
-	)
-	(symbol
 		(lib_id "Device:R")
 		(at 111.76 72.39 180)
@@
 			)
 		)
-		(property "Footprint" "digikey-footprints:TO-92-3"
+		(property "Footprint" "Package_TO_SOT_THT:TO-92_Inline"
 			(at 251.46 66.04 0)
 			(hide yes)
@@
 			)
 		)
-		(property "Value" "MCP4725A0T-ECH"
+		(property "Value" "MCP4726A0T-ECH"
 			(at 175.26 31.75 0)
 			(show_name no)

Commit message: ほぼ完成?
Connections:
- net CAL_MODE: now also U302.19 (IO0); no longer U302.18 (IO1)
- net LOAD: now also U302.18 (IO1); no longer U302.19 (IO0)
- net at Q301.1 (G), R302.2: now also U302.14 (IO5); no longer U302.11 (IO6)
- net at Q302.1 (G), R304.2: now also U302.11 (IO6); no longer U302.14 (IO5)
Changed lines of the file:
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@@
+	(wire
+		(pts
+			(xy 72.39 143.51) (xy 44.45 143.51)
+		)
+		(stroke
+			(width 0)
+			(type default)
+		)
+	)
 	(wire
 		(pts
@@
 	(wire
 		(pts
+			(xy 46.99 140.97) (xy 46.99 179.07)
+		)
+		(stroke
+			(width 0)
+			(type default)
+		)
+	)
+	(wire
+		(pts
 			(xy 62.23 22.86) (xy 66.04 22.86)
 		)
@@
 		(pts
 			(xy 271.78 137.16) (xy 267.97 137.16)
-		)
-		(stroke
-			(width 0)
-			(type default)
-		)
-	)
-	(wire
-		(pts
-			(xy 46.99 143.51) (xy 72.39 143.51)
 		)
 		(stroke
@@
 	(wire
 		(pts
-			(xy 46.99 143.51) (xy 46.99 179.07)
-		)
-		(stroke
-			(width 0)
-			(type default)
-		)
-	)
-	(wire
-		(pts
 			(xy 55.88 44.45) (xy 55.88 45.72)
 		)
@@
 	(wire
 		(pts
+			(xy 46.99 140.97) (xy 72.39 140.97)
+		)
+		(stroke
+			(width 0)
+			(type default)
+		)
+	)
+	(wire
+		(pts
 			(xy 210.82 99.06) (xy 214.63 99.06)
 		)
@@
 		(pts
 			(xy 200.66 57.15) (xy 200.66 58.42)
-		)
-		(stroke
-			(width 0)
-			(type default)
-		)
-	)
-	(wire
-		(pts
-			(xy 44.45 140.97) (xy 44.45 194.31)
 		)
 		(stroke
@@
 	(wire
 		(pts
-			(xy 72.39 140.97) (xy 44.45 140.97)
-		)
-		(stroke
-			(width 0)
-			(type default)
-		)
-	)
-	(wire
-		(pts
 			(xy 105.41 81.28) (xy 121.92 81.28)
 		)
@@
 		(pts
 			(xy 148.59 67.31) (xy 153.67 67.31)
+		)
+		(stroke
+			(width 0)
+			(type default)
+		)
+	)
+	(wire
+		(pts
+			(xy 44.45 143.51) (xy 44.45 194.31)
 		)
 		(stroke
@@
 		)
 	)
+	(label "CAL_MODE"
+		(at 69.85 128.27 180)
+		(effects
+			(font
+				(size 1.27 1.27)
+			)
+			(justify right bottom)
+		)
+	)
 	(label "GAIN_0X"
 		(at 147.32 31.75 0)
@@
 		)
 	)
-	(label "CAL_MODE"
-		(at 69.85 130.81 180)
-		(effects
-			(font
-				(size 1.27 1.27)
-			)
-			(justify right bottom)
-		)
-	)
 	(label "SCL"
 		(at 177.8 101.6 180)
@@
 		)
 	)
-	(label "LOAD"
-		(at 69.85 128.27 180)
-		(effects
-			(font
-				(size 1.27 1.27)
-			)
-			(justify right bottom)
-		)
-	)
 	(label "GAIN_X0"
 		(at 147.32 34.29 0)
@@
 		(effects
 			(font
+				(size 1.27 1.27)
+			)
+			(justify right bottom)
+		)
+	)
+	(label "LOAD"
+		(at 69.85 130.81 180)
+		(effects
+			(font
