File: v2_interface.kicad_sch (KiCad schematic)
At the start: 53 parts, among them J301 BH-14SG, J302 PH-2x3SG, Q301 2N7002K, Q302 2N7002K, Q303 BSS84, Q304 2N7002K, Q305 2N7002K, U301 74LCX541FT, U302 SLG46826G, U303 PCA9515AD, U304 MCP4726A0T-ECH, U305 MCP3424T-ESL, U306 MCP9701A-E_TO

Commit message: できたかも
Parts:
- C301, C302, C303, C304, C305, C306, C309: Akizuki_code2 (none) -> 116143
- D301: Akizuki_code 108275 -> 103982
- D302: Akizuki_code 108275 -> 103978
- D303: Akizuki_code 108275 -> 103980
- Q303: Akizuki_code (none) -> 104269
- R301, R302, R304, R306, R307, R308, R309, R310, R311, R312, R313, R314, R315, R317: Akizuki_code 106668 -> 115029
- R303, R305, R316: Akizuki_code 10668 -> 114122
- R318, R319: Sengoku_code (none) -> EEHD-57HU
- R320, R321, R322, R323, R324: Akizuki_code (none) -> 106201
- TP301: Akizuki_code (none) -> 131773
- U301: Akizuki_code (none) -> 114112
- U302: Akizuki_code (none) -> 118384
- U303: Akizuki_code (none) -> 110882
- U304: Akizuki_code (none) -> 107611
- U305: Akizuki_code (none) -> 111989
- U306: Akizuki_code (none) -> 103199

Commit message: 現状確定
Parts:
- added J303: PH-1X3SG, Connector_PinHeader_2.54mm:PinHeader_1x03_P2.54mm_Vertical, symbol Connector_Generic:Conn_01x03
- added J304: B2B-XH-A, Connector_JST:JST_XH_B2B-XH-A_1x02_P2.50mm_Vertical, symbol Connector_Generic:Conn_01x02
- C301, C302, C303, C304, C305, C306, C309: In_Stock (none) -> 77
- C307, C308, C310, C311, C312, D301, D302, D303, J301, Q303, TP301, U301, U302, U303, U304, U306: In_Stock (none) -> 0
- J302: In_Stock (none) -> (Cut)
- Q301, Q302, Q304, Q305: In_Stock (none) -> 16
- R301, R302, R304, R306, R307, R308, R309, R310, R311, R312, R313, R314, R315, R317, R320, R321, R322, R323, R324: In_Stock (none) -> >100
- R303, R305, R316: In_Stock (none) -> 170
- R318, R319: In_Stock (none) -> 51
- U305: In_Stock (none) -> 1
Connections:
- net GND: now also J304.2 (Pin_2)
- net rt: now also J303.2 (Pin_2); no longer U304.1 (VOUT)
- new net: J303.1 (Pin_1), U304.1 (VOUT)
- new net: J303.3 (Pin_3), J304.1 (Pin_1)
Other:
- moved on the sheet: C301, C302, C303, C304, C305, C306, C307, C308, C309, C310, C311, C312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
