File: Main_SMD_Controller_v2.kicad_pcb (KiCad board)
At the start: 4 copper layers, 100 x 80 mm, 107 parts, among them J1 Sens, J10 Vref_Select, J11 AnalogIO, J12 AUX_Select, J13 DB25_Socket, J14 I^{2}C_TP1, J15 I^{2}C_TP2, J16 SPI_TP1, J17 SPI_TP2, J18 3P_TempSensor, J19 TP, J2 VsensJMP, J20 CS_TP, J21 ModPower, J22 5V_PWR, J23 OP_PWR, J3 Vin+, J4 Drain, J5 Gate, J6 Source, J7 Vin_-, J8 GAIN_TP, J9 MODE_TP, P1 Eoshi-chan_Silk, P2 Eoshi-chan_Silk, P3 Serial_QR, Q1 2N7002K, Q2 2N7002K, U1 OP07, U10 MCP3424x-xSL, U2 ADA4510-2ARZ, U3 AD633ANZ, U4 ADA4522-1ARZ, U5 TC74HC4066AP, U6 TC74HC4066AP, U7 LT1167CN8, U8 MCP4922, U9 MCP1501-20xCH

Commit message: aaaa
Parts:
- removed C1: 0.001u, Capacitor_SMD:C_0603_1608Metric
- removed C10, C11, C17, C18, C19, C20, C21, C22, C23, C4, C5, C6, C7, C8, C9: 0.1u, Capacitor_SMD:C_0603_1608Metric
- removed C12, C14, C16: 100p, Capacitor_SMD:C_0603_1608Metric
- removed C13, C15: 1000p, Capacitor_SMD:C_0603_1608Metric
- removed C2, C3: 0.01u(FL), Capacitor_THT:C_Rect_L7.0mm_W2.5mm_P5.00mm
- removed D1: 1N4007, Diode_THT:D_DO-41_SOD81_P10.16mm_Horizontal
- removed D2: OSR5PA5A33A-1MA, LED_THT:LED_D5.0mm
- removed J1: Sens, Connector_JST:JST_VH_B2P3-VH_1x02_P7.92mm_Vertical
- removed J10: Vref_Select, Connector_PinHeader_2.54mm:PinHeader_1x03_P2.54mm_Vertical
- removed J11: AnalogIO, Connector_PinHeader_2.54mm:PinHeader_2x05_P2.54mm_Vertical
- removed J12: AUX_Select, Connector_PinHeader_2.54mm:PinHeader_1x03_P2.54mm_Vertical
- removed J13: DB25_Socket, AM_Conn_Dsub:Dsub-25P_2.77mm-2.84mm-8.08mmOffset
- removed J14: I^{2}C_TP1, Connector_PinHeader_2.54mm:PinHeader_1x03_P2.54mm_Vertical
- removed J15: I^{2}C_TP2, Connector_PinHeader_2.54mm:PinHeader_1x03_P2.54mm_Vertical
- removed J16: SPI_TP1, Connector_PinHeader_2.54mm:PinHeader_1x04_P2.54mm_Vertical
- removed J17: SPI_TP2, Connector_PinHeader_2.54mm:PinHeader_1x04_P2.54mm_Vertical
- removed J18: 3P_TempSensor, Connector_PinSocket_2.54mm:PinSocket_1x03_P2.54mm_Vertical
- removed J19: TP, Connector_PinHeader_2.54mm:PinHeader_1x03_P2.54mm_Vertical
- removed J2: VsensJMP, Connector_PinHeader_2.54mm:PinHeader_1x03_P2.54mm_Vertical
- removed J20: CS_TP, Connector_PinHeader_2.54mm:PinHeader_1x04_P2.54mm_Vertical
- removed J21: ModPower, Connector_PinHeader_2.00mm:PinHeader_2x02_P2.00mm_Vertical
- removed J22: 5V_PWR, AM_Conn_ScrewTerminal:EurostylePluggable_1x02_P5.08mm
- removed J23: OP_PWR, AM_Conn_ScrewTerminal:EurostylePluggable_1x03_P5.08mm
- removed J3: Vin+, AM_Conn_ScrewTerminal:ScrewTerminal_01x01_PCB-20
- removed J4: Drain, AM_Conn_ScrewTerminal:ScrewTerminal_01x01_PCB-20
- removed J5: Gate, Connector_JST:JST_XH_B2B-XH-A_1x02_P2.50mm_Vertical
- removed J6: Source, AM_Conn_ScrewTerminal:ScrewTerminal_01x01_PCB-20
- removed J7: Vin_-, AM_Conn_ScrewTerminal:ScrewTerminal_01x01_PCB-20
- removed J8: GAIN_TP, Connector_PinHeader_2.54mm:PinHeader_1x04_P2.54mm_Vertical
- removed J9: MODE_TP, Connector_PinHeader_2.54mm:PinHeader_1x04_P2.54mm_Vertical
- removed P1: Eoshi-chan_Silk, Eoshi-chan:Eoshi-chan_logo_15x15
- removed P2: Eoshi-chan_Silk, Eoshi-chan_v2:Eoshi-chan-v2_10x10
- removed P3: Serial_QR, JLCPCB_Serial:Serial_QR_5x5
- removed Q1, Q2: 2N7002K, Package_TO_SOT_SMD:SOT-23
- removed R1: 39k(1), Resistor_THT:R_Axial_DIN0207_L6.3mm_D2.5mm_P2.54mm_Vertical
- removed R10: 33k(1), Resistor_THT:R_Axial_DIN0207_L6.3mm_D2.5mm_P2.54mm_Vertical
- removed R11: 100, Resistor_THT:R_Axial_DIN0207_L6.3mm_D2.5mm_P2.54mm_Vertical
- removed R12, R4, R7, R9: 10k(1), Resistor_THT:R_Axial_DIN0207_L6.3mm_D2.5mm_P2.54mm_Vertical
- removed R13, R15, R16, R17: R(1), Resistor_THT:R_Axial_DIN0207_L6.3mm_D2.5mm_P2.54mm_Vertical
- removed R14: 20m, Resistor_THT:R_Bare_Metal_Element_L16.3mm_W4.8mm_P15.30mm
- removed R18, R19, R22, R23, R24: 200, Resistor_SMD:R_0603_1608Metric
- removed R2: 100k(1%), Resistor_THT:R_Axial_DIN0207_L6.3mm_D2.5mm_P2.54mm_Vertical
- removed R20, R21, R25, R26, R27: 10k, Resistor_SMD:R_0603_1608Metric
- removed R3, R8: 20k(1), Resistor_THT:R_Axial_DIN0207_L6.3mm_D2.5mm_P2.54mm_Vertical
- removed R5: 10k(1%), Resistor_THT:R_Axial_DIN0207_L6.3mm_D2.5mm_P2.54mm_Vertical
- removed R6: 510k(1), Resistor_THT:R_Axial_DIN0207_L6.3mm_D2.5mm_P2.54mm_Vertical
- removed RLY1: 943-1C-5DS, AM_Relay:HSINDA-943_12A-1C_5p
- removed RV1, RV2, RV3, RV4: R_Trim, Potentiometer_THT:Potentiometer_Bourns_3296W_Vertical
- removed TP1: BIAS, TestPoint:TestPoint_Loop_D2.50mm_Drill1.0mm
- removed TP10: ~{LOAD_G}, TestPoint:TestPoint_Loop_D2.50mm_Drill1.0mm
- removed TP2: Vmeas, TestPoint:TestPoint_Loop_D2.50mm_Drill1.0mm
- removed TP3: Pcalc, TestPoint:TestPoint_Loop_D2.50mm_Drill1.0mm
- removed TP4: FeedBack, TestPoint:TestPoint_Loop_D2.50mm_Drill1.0mm
- removed TP5: Set, TestPoint:TestPoint_Loop_D2.50mm_Drill1.0mm
- removed TP7: Imeas, TestPoint:TestPoint_Loop_D2.50mm_Drill1.0mm
- removed TP9: ADC_Vref, TestPoint:TestPoint_Loop_D2.50mm_Drill1.0mm
- removed U1: OP07, Package_DIP:DIP-8_W7.62mm
- removed U10: MCP3424x-xSL, Package_DIP:DIP-14_W7.62mm
- removed U2: ADA4510-2ARZ, Package_DIP:DIP-8_W7.62mm
- removed U3: AD633ANZ, Package_DIP:DIP-8_W7.62mm
- removed U4: ADA4522-1ARZ, Package_DIP:DIP-8_W7.62mm
- removed U5, U6: TC74HC4066AP, Package_DIP:DIP-14_W7.62mm
- removed U7: LT1167CN8, Package_DIP:DIP-8_W7.62mm
- removed U8: MCP4922, Package_DIP:DIP-14_W7.62mm
- removed U9: MCP1501-20xCH, Package_TO_SOT_SMD:SOT-23-6
- added C101: 47u, Capacitor_SMD:CP_Elec_6.3x5.9, F.Cu at (69.8, 127.4)
- added C102: 47u, Capacitor_SMD:CP_Elec_6.3x5.9, F.Cu at (69.8, 135.5)
- added C103: 47u, Capacitor_SMD:CP_Elec_6.3x5.9, F.Cu at (69.8, 143.7)
- added C104: 1u, Capacitor_SMD:C_0603_1608Metric, F.Cu at (50.1, 127.0)
- added C105: 1u, Capacitor_SMD:C_0603_1608Metric, F.Cu at (50.1, 129.5)
- added C106: 1u, Capacitor_SMD:C_0603_1608Metric, F.Cu at (50.1, 132.0)
- added C107: 0.1u, Capacitor_SMD:C_0603_1608Metric, F.Cu at (50.1, 134.5)
- added C108: 0.1u, Capacitor_SMD:C_0603_1608Metric, F.Cu at (50.1, 137.1)
- added C109: 0.1u, Capacitor_SMD:C_0603_1608Metric, F.Cu at (50.1, 139.6)
- added C110: 0.1u, Capacitor_SMD:C_0603_1608Metric, F.Cu at (54.2, 127.0)
- added C111: 0.1u, Capacitor_SMD:C_0603_1608Metric, F.Cu at (54.2, 129.5)
- added C112: 0.1u, Capacitor_SMD:C_0603_1608Metric, F.Cu at (54.2, 132.0)
- added C113: 0.1u, Capacitor_SMD:C_0603_1608Metric, F.Cu at (54.2, 134.5)
- added C114: 4.7u, Capacitor_SMD:C_1210_3225Metric, F.Cu at (108.2, 122.7)
- added C115: 4.7u, Capacitor_SMD:C_1210_3225Metric, F.Cu at (108.2, 126.9)
- added C116: 4.7u, Capacitor_SMD:C_1210_3225Metric, F.Cu at (108.2, 131.2)
- added C117: 0.1u, Capacitor_SMD:C_0603_1608Metric, F.Cu at (54.2, 137.1)
- added C118: 0.1u, Capacitor_SMD:C_0603_1608Metric, F.Cu at (54.2, 139.6)
- added C119: xx, Capacitor_SMD:C_0603_1608Metric, F.Cu at (58.2, 127.0)
- added C120: 0.1u, Capacitor_SMD:C_0603_1608Metric, F.Cu at (58.2, 129.5)
- added C121: 0.1u, Capacitor_SMD:C_0603_1608Metric, F.Cu at (58.2, 132.0)
- added C122: 0.1u, Capacitor_SMD:C_0603_1608Metric, F.Cu at (58.2, 134.5)
- added C123: 0.1u, Capacitor_SMD:C_0603_1608Metric, F.Cu at (58.2, 137.1)
- added C124: 0.1u, Capacitor_SMD:C_0603_1608Metric, F.Cu at (58.2, 139.6)
- added C125: xx, Capacitor_SMD:C_0603_1608Metric, F.Cu at (62.2, 127.0)
- added C126: 0.1u, Capacitor_SMD:C_0603_1608Metric, F.Cu at (62.2, 129.5)
- added C127: 0.1u, Capacitor_SMD:C_0603_1608Metric, F.Cu at (62.2, 132.0)
- added C201: 0.1u, Capacitor_SMD:C_0603_1608Metric, F.Cu at (55.6, 152.2)
- added C202: 0.1u, Capacitor_SMD:C_0603_1608Metric, F.Cu at (55.6, 154.7)
- added C203: xx, Capacitor_SMD:C_0603_1608Metric, F.Cu at (55.6, 157.2)
- added C204: 0.01u(FL), Capacitor_SMD:C_0805_2012Metric, F.Cu at (69.8, 173.1)
- added C205: 0.1u, Capacitor_SMD:C_0603_1608Metric, F.Cu at (55.6, 159.7)
- added C206: xx, Capacitor_SMD:C_0603_1608Metric, F.Cu at (55.6, 162.2)
- added C207: 0.1u, Capacitor_SMD:C_0603_1608Metric, F.Cu at (55.6, 164.7)
- added C208: 1000p, Capacitor_SMD:C_0805_2012Metric, F.Cu at (69.8, 176.1)
- added C209: 10p, Capacitor_SMD:C_0603_1608Metric, F.Cu at (59.6, 152.2)
- added C210: 0.047u(FL), Capacitor_THT:C_Rect_L7.2mm_W5.0mm_P5.00mm, F.Cu at (43.9, 178.0)
- added C301: 0.1u, Capacitor_SMD:C_0603_1608Metric, F.Cu at (78.1, 152.2)
- added C302: 0.1u, Capacitor_SMD:C_0603_1608Metric, F.Cu at (78.1, 154.7)
- added C303: 1000p, Capacitor_SMD:C_0603_1608Metric, F.Cu at (78.1, 157.2)
- added C304: 1000p, Capacitor_SMD:C_0603_1608Metric, F.Cu at (78.1, 159.7)
- added C305: 1000p, Capacitor_SMD:C_0603_1608Metric, F.Cu at (78.1, 162.2)
- added C306: 1000p, Capacitor_SMD:C_0603_1608Metric, F.Cu at (78.1, 164.7)
- added C307: 1000p, Capacitor_SMD:C_0603_1608Metric, F.Cu at (82.1, 152.2)
- added D101: GS1010FL, Diode_SMD:D_SOD-123F, F.Cu at (97.8, 138.3)
- added D301: OSG50603C1E, LED_SMD:LED_0603_1608Metric, F.Cu at (83.1, 171.9)
- added FB101: BLM21PG331SN, Inductor_SMD:L_0805_2012Metric, F.Cu at (108.6, 99.1)
- added FB102: BLM21PG331SN, Inductor_SMD:L_0805_2012Metric, F.Cu at (108.6, 101.9)
- added FB103: BLM21PG331SN, Inductor_SMD:L_0805_2012Metric, F.Cu at (108.6, 104.6)
- added FB104: BLM21PG331SN, Inductor_SMD:L_0805_2012Metric, F.Cu at (108.6, 107.4)
- added J101: B3B-XH-A, AM_Conn_ScrewTerminal:EurostylePluggable_1x03_P5.08mm, F.Cu at (56.3, 111.0)
- added J102: B3B-XH-A, AM_Conn_ScrewTerminal:EurostylePluggable_1x03_P5.08mm, F.Cu at (56.3, 125.0)
- added J103: B2B-XH-A, Connector_JST:JST_XH_B2B-XH-A_1x02_P2.50mm_Vertical, F.Cu at (99.4, 123.9)
- added J104: B2B-XH-A, Connector_JST:JST_XH_B2B-XH-A_1x02_P2.50mm_Vertical, F.Cu at (99.4, 131.7)
- added J105: PH-1X3SG, Connector_PinHeader_2.54mm:PinHeader_1x03_P2.54mm_Vertical, F.Cu at (107.0, 85.3)
- added J106: PCB-20, AM_Conn_ScrewTerminal:ScrewTerminal_01x01_PCB-20, F.Cu at (47.9, 90.4)
- added J107: PCB-20, AM_Conn_ScrewTerminal:ScrewTerminal_01x01_PCB-20, F.Cu at (59.6, 90.4)
- added J108: PCB-20, AM_Conn_ScrewTerminal:ScrewTerminal_01x01_PCB-20, F.Cu at (71.3, 90.4)
- added J109: PCB-20, AM_Conn_ScrewTerminal:ScrewTerminal_01x01_PCB-20, F.Cu at (83.0, 90.4)
- added J302: PH-2x3SG, Connector_PinHeader_2.54mm:PinHeader_2x03_P2.54mm_Vertical, F.Cu at (90.4, 163.6)
- added P101: Eoshi-chan_Silk, Eoshi-chan:Eoshi-chan_logo_15x15, F.Cu at (96.8, 89.5)
- added P102: Eoshi-chan_Silk, Eoshi-chan_v2:Eoshi-chan-v2_10x10, F.Cu at (101.4, 144.7)
- added P103: Serial_QR, JLCPCB_Serial:Serial_QR_5x5, F.Cu at (79.6, 143.9)
- added Q201: 2SC1815, Package_TO_SOT_THT:TO-92L_Inline, F.Cu at (69.6, 169.2)
- added Q202: 2SD1415A, Package_TO_SOT_THT:TO-220-3_Vertical, F.Cu at (45.2, 154.8)
- added Q203: TTB1020B, Package_TO_SOT_THT:TO-220-3_Vertical, F.Cu at (45.2, 160.8)
- added Q204: 2SD1415A, Package_TO_SOT_THT:TO-220-3_Vertical, F.Cu at (45.2, 166.7)
- added Q205: TTB1020B, Package_TO_SOT_THT:TO-220-3_Vertical, F.Cu at (45.2, 172.7)
- added Q301: 2N7002K, Package_TO_SOT_SMD:SOT-23, F.Cu at (78.6, 168.2)
- added Q302: 2N7002K, Package_TO_SOT_SMD:SOT-23, F.Cu at (78.6, 172.6)
- added R101: 100k(0.1), Resistor_SMD:R_0805_2012Metric, F.Cu at (93.7, 122.0)
- added R102: 10k(0.1), Resistor_SMD:R_0805_2012Metric, F.Cu at (93.7, 125.0)
- added R103: 1k(0.1), Resistor_SMD:R_0805_2012Metric, F.Cu at (93.7, 127.9)
- added R104: 100, Resistor_SMD:R_0603_1608Metric, F.Cu at (62.2, 134.5)
- added R105: 10k(0.1), Resistor_SMD:R_0805_2012Metric, F.Cu at (93.7, 130.9)
- added R106: 2.2k(0.5), Resistor_THT:R_Axial_DIN0207_L6.3mm_D2.5mm_P2.54mm_Vertical, F.Cu at (44.0, 99.8)
- added R107: 10k(0.1), Resistor_SMD:R_0805_2012Metric, F.Cu at (93.7, 133.8)
- added R108: 1k(0.1), Resistor_SMD:R_0805_2012Metric, F.Cu at (93.7, 136.8)
- added R109: 39k(0.5), Resistor_THT:R_Axial_DIN0207_L6.3mm_D2.5mm_P2.54mm_Vertical, F.Cu at (44.0, 103.8)
- added R110: 1k(0.5), Resistor_THT:R_Axial_DIN0207_L6.3mm_D2.5mm_P2.54mm_Vertical, F.Cu at (44.0, 107.9)
- added R111: R(0.5), Resistor_THT:R_Axial_DIN0207_L6.3mm_D2.5mm_P2.54mm_Vertical, F.Cu at (44.0, 111.9)
- added R112: R(0.5), Resistor_THT:R_Axial_DIN0207_L6.3mm_D2.5mm_P2.54mm_Vertical, F.Cu at (44.0, 116.0)
- added R113: R(0.5), Resistor_THT:R_Axial_DIN0207_L6.3mm_D2.5mm_P2.54mm_Vertical, F.Cu at (44.0, 120.0)
- added R114: R(0.5), Resistor_THT:R_Axial_DIN0207_L6.3mm_D2.5mm_P2.54mm_Vertical, F.Cu at (44.0, 124.1)
- added R115: BR3FB10L0 (10m), Resistor_THT:R_Bare_Metal_Element_L16.3mm_W4.8mm_P15.30mm, F.Cu at (77.8, 117.4)
- added R201: 10k, Resistor_SMD:R_0603_1608Metric, F.Cu at (59.6, 154.7)
- added R202: 0, Resistor_SMD:R_0603_1608Metric, F.Cu at (59.6, 157.2)
- added R203: 1k, Resistor_SMD:R_0603_1608Metric, F.Cu at (59.6, 159.7)
- added R204: 0, Resistor_SMD:R_0603_1608Metric, F.Cu at (59.6, 162.2)
- added R205: 0, Resistor_SMD:R_0603_1608Metric, F.Cu at (59.6, 164.7)
- added R206: 10k, Resistor_SMD:R_0603_1608Metric, F.Cu at (63.6, 152.2)
- added R207: 100k, Resistor_SMD:R_0603_1608Metric, F.Cu at (63.6, 154.7)
- added R208: 510, Resistor_SMD:R_1206_3216Metric, F.Cu at (68.4, 159.1)
- added R209: 3k, Resistor_SMD:R_0603_1608Metric, F.Cu at (63.6, 157.2)
- added R210: 1k, Resistor_SMD:R_0805_2012Metric, F.Cu at (65.4, 167.4)
- added R211: 510, Resistor_SMD:R_1206_3216Metric, F.Cu at (68.4, 162.5)
- added R212: 470, Resistor_SMD:R_0805_2012Metric, F.Cu at (65.4, 170.4)
- added R213: 470, Resistor_SMD:R_0805_2012Metric, F.Cu at (65.4, 173.3)
- added R214: 1k, Resistor_SMD:R_0603_1608Metric, F.Cu at (63.6, 159.7)
- added R217: 470, Resistor_SMD:R_0805_2012Metric, F.Cu at (65.4, 176.3)
- added R218: 470, Resistor_SMD:R_0805_2012Metric, F.Cu at (65.4, 179.2)
- added R221: 4.7, Resistor_SMD:R_2512_6332Metric, F.Cu at (57.9, 179.0)
- added R301: 10k, Resistor_SMD:R_0603_1608Metric, F.Cu at (82.1, 154.7)
- added R302: 10k, Resistor_SMD:R_0603_1608Metric, F.Cu at (82.1, 157.2)
- added R303: 10k, Resistor_SMD:R_0603_1608Metric, F.Cu at (82.1, 159.7)
- added R304: 1k, Resistor_SMD:R_0603_1608Metric, F.Cu at (82.1, 162.2)
- added R305: 200, Resistor_SMD:R_0603_1608Metric, F.Cu at (82.1, 164.7)
- added R306: 200, Resistor_SMD:R_0603_1608Metric, F.Cu at (86.1, 152.2)
- added R307: 200, Resistor_SMD:R_0603_1608Metric, F.Cu at (86.1, 154.7)
- added R308: 200, Resistor_SMD:R_0603_1608Metric, F.Cu at (86.1, 157.2)
- added R309: 200, Resistor_SMD:R_0603_1608Metric, F.Cu at (86.1, 159.7)
- added R310: 10k, Resistor_SMD:R_0603_1608Metric, F.Cu at (86.1, 162.2)
- added RLY101: 943-1C-5DS, AM_Relay:HSINDA-943_12A-1C_5p, F.Cu at (85.6, 106.0)
- added RV101: R_Trim, Potentiometer_THT:Potentiometer_Bourns_3296W_Vertical, F.Cu at (72.6, 100.9)
- added RV102: R_Trim, Potentiometer_THT:Potentiometer_Bourns_3296W_Vertical, F.Cu at (72.6, 107.3)
- added RV103: R_Trim, Potentiometer_THT:Potentiometer_Bourns_3296W_Vertical, F.Cu at (72.6, 113.7)
- added RV104: R_Trim, Potentiometer_THT:Potentiometer_Bourns_3296W_Vertical, F.Cu at (72.6, 120.1)
- added RV201: 2k, AM_Potentiometer:TSR-065-xxx-R, F.Cu at (55.9, 173.8)
- added U101: XC6201P332MR-G, Package_TO_SOT_SMD:SOT-23-5, F.Cu at (88.9, 122.9)
- added U102: XC6902N331MR-G, Package_TO_SOT_SMD:SOT-23-3, F.Cu at (59.2, 143.0)
- added U103: XC6201P502MR-G, Package_TO_SOT_SMD:SOT-23-5, F.Cu at (88.9, 127.6)
- added U104: MCP1501-20E/CHY, Package_TO_SOT_SMD:SOT-23-6, F.Cu at (88.9, 132.2)
- added U105: ADA4510-2ARZ, Package_SO:SOIC-8_3.9x4.9mm_P1.27mm, F.Cu at (52.4, 144.2)
- added U106: NJU7098A, Package_TO_SOT_SMD:SOT-23-6, F.Cu at (88.9, 136.8)
- added U107: TC4066BP, Package_DIP:DIP-14_W7.62mm, F.Cu at (77.2, 122.6)
- added U108: LT1167CN8, Package_DIP:DIP-8_W7.62mm, F.Cu at (97.2, 99.8)
- added U201: ADA4522-1ARZ, Package_SO:SOIC-8_3.9x4.9mm_P1.27mm, F.Cu at (69.8, 154.3)
- added U202: KIA75S358F, Package_TO_SOT_SMD:SOT-23-5, F.Cu at (70.1, 180.0)
- added U301: MCP4725A0T-ECH, Package_TO_SOT_SMD:SOT-23-6, F.Cu at (83.6, 168.4)
- added U302: MCP3424x-xSL, Package_SO:SOIC-14_3.9x8.7mm_P1.27mm, F.Cu at (92.4, 156.2)
- renumbered H1 to H101, H2 to H102, H3 to H103, H4 to H104
Routing:
- net +5V: track 252.1 -> 0.00 mm
- net GNDA: track 189.7 -> 0.00 mm
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- removed copper zone on B.Cu, net GND
- removed copper zone on F.Cu, net GND

Commit message: kannsei
Parts:
- removed C124, C126, C127: 0.1u, Capacitor_SMD:C_0603_1608Metric
- removed C125: xx, Capacitor_SMD:C_0603_1608Metric
- removed P103: Serial_QR, JLCPCB_Serial:Serial_QR_5x5
- removed U108: LT1167CN8, Package_DIP:DIP-8_W7.62mm
- added C211: 0.1u, Capacitor_SMD:C_0603_1608Metric, F.Cu at (239.7, 111.3)
- added C212: 1000p, Capacitor_SMD:C_0805_2012Metric, F.Cu at (251.5, 90.3)
- added C213: 10p, Capacitor_SMD:C_0603_1608Metric, F.Cu at (239.7, 113.8)
- added C214: 0.047u(FL), Capacitor_THT:C_Rect_L7.2mm_W5.0mm_P5.00mm, F.Cu at (255.6, 87.6)
- added C308: 1000p, Capacitor_SMD:C_0603_1608Metric, F.Cu at (236.1, 135.9)
- added C309: 0.1u, Capacitor_SMD:C_0603_1608Metric, F.Cu at (236.1, 138.4)
- added C310: 1000p, Capacitor_SMD:C_0603_1608Metric, F.Cu at (240.1, 118.3)
- added C311: 1000p, Capacitor_SMD:C_0603_1608Metric, F.Cu at (240.1, 120.8)
- added C312: 1000p, Capacitor_SMD:C_0603_1608Metric, F.Cu at (240.1, 123.3)
- added D302: OSHR1608C1A, LED_SMD:LED_0603_1608Metric, F.Cu at (257.1, 121.0)
- added D303: OSYG1608, LED_SMD:LED_0603_1608Metric, F.Cu at (257.1, 123.5)
- added J110: PCB-20, AM_Conn_ScrewTerminal:ScrewTerminal_01x01_PCB-20, F.Cu at (142.5, 66.5)
- added J301: BH-14SG, Connector_IDC:IDC-Header_2x07_P2.54mm_Vertical, F.Cu at (227.4, 123.2)
- added Q303: BSS84, Package_TO_SOT_SMD:SOT-23, F.Cu at (252.6, 128.2)
- added Q304: 2N7002K, Package_TO_SOT_SMD:SOT-23, F.Cu at (252.6, 132.6)
- added Q305: 2N7002K, Package_TO_SOT_SMD:SOT-23, F.Cu at (252.6, 137.1)
- added R116: BR3FB10L0 (10m), Resistor_THT:R_Bare_Metal_Element_L16.3mm_W4.8mm_P15.30mm, F.Cu at (130.0, 82.7)
- added R215: 470, Resistor_SMD:R_1206_3216Metric, F.Cu at (261.2, 99.2)
- added R216: 470, Resistor_SMD:R_1206_3216Metric, F.Cu at (261.2, 102.5)
- added R219: 1, Resistor_THT:R_Box_L14.0mm_W5.0mm_P9.00mm, F.Cu at (225.4, 83.5)
- added R220: 470, Resistor_SMD:R_1206_3216Metric, F.Cu at (261.2, 105.8)
- added R222: 1, Resistor_THT:R_Box_L14.0mm_W5.0mm_P9.00mm, F.Cu at (225.4, 90.1)
- added R223: 1, Resistor_THT:R_Box_L14.0mm_W5.0mm_P9.00mm, F.Cu at (225.4, 96.6)
- added R224: 4.7, Resistor_SMD:R_2512_6332Metric, F.Cu at (254.1, 109.8)
- added R311: 10k, Resistor_SMD:R_0603_1608Metric, F.Cu at (244.2, 128.4)
- added R312: 10k, Resistor_SMD:R_0603_1608Metric, F.Cu at (244.2, 130.9)
- added R313: 10k, Resistor_SMD:R_0603_1608Metric, F.Cu at (244.2, 133.4)
- added R314: 10k, Resistor_SMD:R_0603_1608Metric, F.Cu at (244.2, 135.9)
- added R315: 10k, Resistor_SMD:R_0603_1608Metric, F.Cu at (244.2, 138.4)
- added R316: 1k, Resistor_SMD:R_0603_1608Metric, F.Cu at (248.2, 118.3)
- added R317: 10k, Resistor_SMD:R_0603_1608Metric, F.Cu at (248.2, 120.8)
- added R318: 0, Resistor_SMD:R_0805_2012Metric, F.Cu at (253.9, 150.8)
- added R319: 0, Resistor_SMD:R_0805_2012Metric, F.Cu at (253.9, 153.8)
- added R320: 200, Resistor_SMD:R_0603_1608Metric, F.Cu at (248.2, 123.3)
- added R321: 200, Resistor_SMD:R_0603_1608Metric, F.Cu at (248.2, 125.9)
- added R322: 200, Resistor_SMD:R_0603_1608Metric, F.Cu at (248.2, 128.4)
- added R323: 200, Resistor_SMD:R_0603_1608Metric, F.Cu at (248.2, 130.9)
- added R324: 200, Resistor_SMD:R_0603_1608Metric, F.Cu at (248.2, 133.4)
- added TP101: RCTCTE, AM_Conn_TP:RCTCE, F.Cu at (212.2, 75.1)
- added TP102: RCTCTE, AM_Conn_TP:RCTCE, F.Cu at (212.2, 77.9)
- added TP103: RCTCTE, AM_Conn_TP:RCTCE, F.Cu at (212.2, 80.7)
- added TP104: RCTCTE, AM_Conn_TP:RCTCE, F.Cu at (212.2, 83.5)
- added TP201: RCTCTE, AM_Conn_TP:RCTCE, F.Cu at (224.0, 101.3)
- added TP202: RCTCTE, AM_Conn_TP:RCTCE, F.Cu at (224.0, 104.1)
- added TP203: RCTCTE, AM_Conn_TP:RCTCE, F.Cu at (224.0, 106.9)
- added TP301: RCTCTE, AM_Conn_TP:RCTCE, F.Cu at (229.1, 152.5)
- added U303: PCA9515AD, Package_SO:SOIC-8_3.9x4.9mm_P1.27mm, F.Cu at (226.4, 147.9)
- added U304: MCP4725A0T-ECH, Package_TO_SOT_SMD:SOT-23-6, F.Cu at (224.7, 153.5)
- added U305: MCP3424T-ESL, Package_SO:SOIC-14_3.9x8.7mm_P1.27mm, F.Cu at (247.5, 144.9)
- added U306: MCP9701A-E_TO, digikey-footprints:TO-92-3, F.Cu at (245.4, 153.0)
- C101, C102, C103: value 47u -> 0.1u; footprint Capacitor_SMD:CP_Elec_6.3x5.9 -> Capacitor_SMD:C_0603_1608Metric
- C104: value 1u -> 0.1u
- C105, C106: value 1u -> 47u; footprint Capacitor_SMD:C_0603_1608Metric -> Capacitor_SMD:CP_Elec_6.3x5.9
- C107, C108: value 0.1u -> 1u
- C111, C112: value 0.1u -> 4.7u; footprint Capacitor_SMD:C_0603_1608Metric -> Capacitor_SMD:C_1210_3225Metric
- C114, C115, C116: value 4.7u -> 0.1u; footprint Capacitor_SMD:C_1210_3225Metric -> Capacitor_SMD:C_0603_1608Metric
- C118, C121: value 0.1u -> NC
- C119: value xx -> 0.1u
- C203: value xx -> 0.01u(FL); footprint Capacitor_SMD:C_0603_1608Metric -> Capacitor_SMD:C_0805_2012Metric
- C204: value 0.01u(FL) -> NC; footprint Capacitor_SMD:C_0805_2012Metric -> Capacitor_SMD:C_0603_1608Metric
- C205: value 0.1u -> NC; footprint Capacitor_SMD:C_0603_1608Metric -> Capacitor_SMD:C_0805_2012Metric
- C206: value xx -> NC; footprint Capacitor_SMD:C_0603_1608Metric -> Capacitor_SMD:C_0805_2012Metric
- C207: value 0.1u -> 1000p(FL); footprint Capacitor_SMD:C_0603_1608Metric -> Capacitor_SMD:C_0805_2012Metric
- C208: value 1000p -> 1000p(FL)
- C209: value 10p -> NC
- C210: value 0.047u(FL) -> 0.1u; footprint Capacitor_THT:C_Rect_L7.2mm_W5.0mm_P5.00mm -> Capacitor_SMD:C_0603_1608Metric
- C303, C304, C305, C306: value 1000p -> 0.1u
- D301: value OSG50603C1E -> OSBL1608C1A
- J101, J102: value B3B-XH-A -> ETB43034G000Z
- J104: value B2B-XH-A -> PH-1X3SG; footprint Connector_JST:JST_XH_B2B-XH-A_1x02_P2.50mm_Vertical -> Connector_PinHeader_2.54mm:PinHeader_1x03_P2.54mm_Vertical
- J105: value PH-1X3SG -> PCB-20; footprint Connector_PinHeader_2.54mm:PinHeader_1x03_P2.54mm_Vertical -> AM_Conn_ScrewTerminal:ScrewTerminal_01x01_PCB-20
- J106: value PCB-20 -> B2B-XH-A; footprint AM_Conn_ScrewTerminal:ScrewTerminal_01x01_PCB-20 -> Connector_JST:JST_XH_B2B-XH-A_1x02_P2.50mm_Vertical
- J108: value PCB-20 -> PH-1X2SG; footprint AM_Conn_ScrewTerminal:ScrewTerminal_01x01_PCB-20 -> Connector_PinHeader_2.54mm:PinHeader_1x02_P2.54mm_Vertical
- P101: footprint Eoshi-chan:Eoshi-chan_logo_15x15 -> Eoshi-chan_v2:Eoshi-chan-v2_10x10
- P102: value Eoshi-chan_Silk -> Serial_QR; footprint Eoshi-chan_v2:Eoshi-chan-v2_10x10 -> JLCPCB_Serial:Serial_QR_5x5
- R101: value 100k(0.1) -> 1k(0.1)
- R102, R105: value 10k(0.1) -> R(0.5); footprint Resistor_SMD:R_0805_2012Metric -> Resistor_THT:R_Axial_DIN0207_L6.3mm_D2.5mm_P2.54mm_Vertical
- R103: value 1k(0.1) -> R(0.5); footprint Resistor_SMD:R_0805_2012Metric -> Resistor_THT:R_Axial_DIN0207_L6.3mm_D2.5mm_P2.54mm_Vertical
- R104: value 100 -> R(0.5); footprint Resistor_SMD:R_0603_1608Metric -> Resistor_THT:R_Axial_DIN0207_L6.3mm_D2.5mm_P2.54mm_Vertical
- R106: value 2.2k(0.5) -> 10k(0.1); footprint Resistor_THT:R_Axial_DIN0207_L6.3mm_D2.5mm_P2.54mm_Vertical -> Resistor_SMD:R_0805_2012Metric
- R107: value 10k(0.1) -> 2.2k(0.5); footprint Resistor_SMD:R_0805_2012Metric -> Resistor_THT:R_Axial_DIN0207_L6.3mm_D2.5mm_P2.54mm_Vertical
- R108: value 1k(0.1) -> 10k(0.1)
- R109: value 39k(0.5) -> 1k(0.1); footprint Resistor_THT:R_Axial_DIN0207_L6.3mm_D2.5mm_P2.54mm_Vertical -> Resistor_SMD:R_0805_2012Metric
- R110: value 1k(0.5) -> 39k(0.5)
- R111: value R(0.5) -> 1k(0.5)
- R112: value R(0.5) -> 100k(0.1); footprint Resistor_THT:R_Axial_DIN0207_L6.3mm_D2.5mm_P2.54mm_Vertical -> Resistor_SMD:R_0805_2012Metric
- R113: value R(0.5) -> 10k(0.1); footprint Resistor_THT:R_Axial_DIN0207_L6.3mm_D2.5mm_P2.54mm_Vertical -> Resistor_SMD:R_0805_2012Metric
- R114: value R(0.5) -> 0; footprint Resistor_THT:R_Axial_DIN0207_L6.3mm_D2.5mm_P2.54mm_Vertical -> Resistor_SMD:R_0805_2012Metric
- R115: value BR3FB10L0 (10m) -> 100; footprint Resistor_THT:R_Bare_Metal_Element_L16.3mm_W4.8mm_P15.30mm -> Resistor_SMD:R_0603_1608Metric
- R201, R303: value 10k -> 1k
- R203: value 1k -> 1M
- R204: value 0 -> 1M
- R205: value 0 -> NC
- R206: value 10k -> 0
- R207: value 100k -> 0
- R208: value 510 -> 10k; footprint Resistor_SMD:R_1206_3216Metric -> Resistor_SMD:R_0603_1608Metric
- R209: value 3k -> 100k
- R210: value 1k -> 3.3k; footprint Resistor_SMD:R_0805_2012Metric -> Resistor_SMD:R_0603_1608Metric
- R211: footprint Resistor_SMD:R_1206_3216Metric -> Resistor_SMD:R_2512_6332Metric
- R212: value 470 -> 1k
- R213: value 470 -> 510; footprint Resistor_SMD:R_0805_2012Metric -> Resistor_SMD:R_2512_6332Metric
- R214: value 1k -> 33k
- R217: value 470 -> 1k; footprint Resistor_SMD:R_0805_2012Metric -> Resistor_SMD:R_0603_1608Metric
- R218: value 470 -> 1; footprint Resistor_SMD:R_0805_2012Metric -> Resistor_THT:R_Box_L14.0mm_W5.0mm_P9.00mm
- R221: value 4.7 -> 470; footprint Resistor_SMD:R_2512_6332Metric -> Resistor_SMD:R_1206_3216Metric
- R304: value 1k -> 10k
- R305: value 200 -> 1k
- R306, R307, R308, R309: value 200 -> 10k
- U103: value XC6201P502MR-G -> TC4066BP; footprint Package_TO_SOT_SMD:SOT-23-5 -> Package_DIP:DIP-14_W7.62mm
- U104: value MCP1501-20E/CHY -> ADA4510-2ARZ; footprint Package_TO_SOT_SMD:SOT-23-6 -> Package_SO:SOIC-8_3.9x4.9mm_P1.27mm
- U105: value ADA4510-2ARZ -> MCP1501-20E/CHY; footprint Package_SO:SOIC-8_3.9x4.9mm_P1.27mm -> Package_TO_SOT_SMD:SOT-23-6
- U106: value NJU7098A -> LT1167CN8; footprint Package_TO_SOT_SMD:SOT-23-6 -> Package_DIP:DIP-8_W7.62mm
- U107: value TC4066BP -> NJU7098A; footprint Package_DIP:DIP-14_W7.62mm -> Package_TO_SOT_SMD:SOT-23-6
- U301: value MCP4725A0T-ECH -> 74LCX541FT; footprint Package_TO_SOT_SMD:SOT-23-6 -> Package_SO:TSSOP-20_4.4x6.5mm_P0.65mm
- U302: value MCP3424x-xSL -> SLG46826G; footprint Package_SO:SOIC-14_3.9x8.7mm_P1.27mm -> Package_SO:TSSOP-20_4.4x6.5mm_P0.65mm
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Connections:
- C101 pad 1: +5V -> Net-(J101-Pin_1)
- C102 pad 2: -5V -> Net-(J101-Pin_3)
- C103 pad 1: +12V -> Net-(J102-Pin_1)
- C104 pad 1: +5V -> GND
- C104 pad 2: GND -> Net-(J102-Pin_3)
- C105 pad 1: -5V -> +5V
- C106 pad 1: +12V -> GND
- C106 pad 2: GND -> -5V
- C107 pad 1: Net-(J101-Pin_1) -> +5V
- C108 pad 1: GND -> -5V
- C108 pad 2: Net-(J101-Pin_3) -> GND
- C109 pad 1: Net-(J102-Pin_1) -> +3V3
- C110 pad 2: Net-(J102-Pin_3) -> -3V3
- C112 pad 1: GND -> -3V3
- C112 pad 2: -3V3 -> GND
- C113 pad 1: +5VA -> +3V3
- C114 pad 1: +3V3 -> -3V3
- C115 pad 1: -3V3 -> +3V3
- C116 pad 1: +5VA -> +3V3
- C117 pad 1: +3V3 -> -3V3
- C118 pad 1: +3V3 -> /Vin
- C118 pad 2: GND -> GNDA
- C119 pad 1: Net-(C119-Pad1) -> +3V3
- C121 pad 1: +3V3 -> Net-(C121-Pad1)
- C122 pad 1: -3V3 -> +3V3
- C123 pad 1: +3V3 -> -3V3
- C201 pad 1: VCC -> +3V3
- C202 pad 1: VEE -> -3V3
- C203 pad 1: Net-(C203-Pad1) -> /Imeas
- C203 pad 2: GND -> Net-(C203-Pad2)
- C204 pad 2: Net-(C204-Pad2) -> GND
- C205 pad 1: +5V -> Net-(C203-Pad2)
- C205 pad 2: GND -> Net-(C205-Pad2)
- C206 pad 1: Net-(C206-Pad1) -> Net-(C203-Pad2)
- C206 pad 2: GND -> Net-(C205-Pad2)
- C207 pad 1: -5V -> Net-(C207-Pad1)
- C207 pad 2: GND -> Net-(C205-Pad2)
- C208 pad 1: Net-(C208-Pad1) -> Net-(C207-Pad1)
- C208 pad 2: Net-(Q201-C) -> Net-(C205-Pad2)
- C209 pad 1: Net-(C208-Pad1) -> Net-(C209-Pad1)
- C209 pad 2: /MOS_G -> GND
- C210 pad 1: Net-(C210-Pad1) -> +5V
- C301 pad 1: +5VA -> +3V3
- C301 pad 2: GND -> GNDD
- C302 pad 1: +5VA -> +3V3
- C302 pad 2: GND -> GNDD
- C303 pad 1: /Interface/Imeas+ -> +3V3
- C303 pad 2: GND -> GNDD
- C304 pad 1: /Interface/Vmeas+ -> +3V3
- C304 pad 2: GND -> GNDD
- C305 pad 1: /Interface/Imeas- -> +3V3
- C306 pad 1: /Interface/Vmeas- -> +3V3
- C307 pad 1: /Interface/OFSmeas -> /Interface/Imeas+
- D101 pad 2: /LOAD_EN -> /RLY_LOUT
- FB101 pad 2: +5V -> +12V
- FB102 pad 2: -5V -> -12V
- FB103 pad 2: +12V -> +5V
- FB104 pad 2: -12V -> -5V
- J103 pad 1: /MOS_G -> Net-(J103-Pin_1)
- J103 pad 2: GND -> GNDA
- J104 pad 1: Net-(J104-Pin_1) -> Net-(J103-Pin_1)
- J104 pad 2: GNDA -> Net-(J104-Pin_2)
- J105 pad 1: Net-(J104-Pin_1) -> /MOS_D
- J106 pad 1: /MOS_D -> /MOS_G
- J108 pad 1: /Load+ -> /OFS
- J109 pad 1: GNDA -> /Load+
- J302 pad 1: /Interface/I^{2}C_SCL -> /Interface/SCL
- J302 pad 2: /Interface/I^{2}C_SCL -> /Interface/SCL
- J302 pad 3: /Interface/I^{2}C_SDA -> /Interface/SDA
- J302 pad 4: /Interface/I^{2}C_SDA -> /Interface/SDA
- J302 pad 5: GND -> GNDD
- J302 pad 6: GND -> GNDD
- Q301 pad 1: /Interface/~{LOAD_G} -> Net-(Q301-G)
- Q301 pad 2: GND -> GNDD
- Q302 pad 1: /Interface/~{LOAD_G} -> Net-(Q302-G)
- Q302 pad 2: GND -> GNDD
- Q302 pad 3: /LOAD_EN -> Net-(D302-K)
- R101 pad 1: Net-(U104-OUT) -> /Vmeas
- R101 pad 2: Net-(C119-Pad1) -> Net-(R101-Pad2)
- R102 pad 1: GND -> Net-(R102-Pad1)
- R102 pad 2: Net-(C119-Pad1) -> Net-(R102-Pad2)
- R103 pad 1: /Vmeas -> Net-(R103-Pad1)
- R104 pad 2: /OFS -> Net-(R104-Pad2)
- R105 pad 1: Net-(R103-Pad2) -> Net-(R105-Pad1)
- R106 pad 1: Net-(R103-Pad2) -> Net-(R101-Pad2)
- R107 pad 1: Net-(R105-Pad2) -> Net-(R101-Pad2)
- R107 pad 2: Net-(R106-Pad2) -> Net-(R107-Pad2)
- R108 pad 2: /OFS -> Net-(R107-Pad2)
- R109 pad 1: Net-(J105-Pin_2) -> Net-(R107-Pad2)
- R109 pad 2: /Vin -> /OFS
- R110 pad 1: GNDA -> Net-(J104-Pin_2)
- R111 pad 1: Net-(R111-Pad1) -> GNDA
- R111 pad 2: Net-(R111-Pad2) -> /Vin
- R112 pad 1: Net-(R112-Pad1) -> Net-(U105-OUT)
- R112 pad 2: Net-(R112-Pad2) -> Net-(C121-Pad1)
- R113 pad 1: Net-(R113-Pad1) -> GND
- R113 pad 2: Net-(R113-Pad2) -> Net-(C121-Pad1)
- R114 pad 1: Net-(R114-Pad1) -> GNDA
- R114 pad 2: Net-(R114-Pad2) -> GND
- R115 pad 1: /MOS_S -> Net-(R115-Pad1)
- R115 pad 2: GNDA -> /OFS
- R201 pad 2: Net-(C204-Pad1) -> Net-(C203-Pad2)
- R202 pad 2: Net-(C203-Pad1) -> Net-(C204-Pad1)
- R203 pad 1: Net-(C204-Pad1) -> Net-(C203-Pad2)
- R203 pad 2: Net-(C204-Pad2) -> Net-(C207-Pad1)
- R204 pad 1: Net-(C204-Pad2) -> Net-(C203-Pad2)
- R204 pad 2: Net-(R204-Pad2) -> Net-(C207-Pad1)
- R205 pad 1: Net-(R204-Pad2) -> Net-(C203-Pad2)
- R205 pad 2: Net-(C206-Pad1) -> Net-(C205-Pad2)
- R206 pad 1: Net-(C206-Pad1) -> Net-(C205-Pad2)
- R206 pad 2: GND -> Net-(R206-Pad2)
- R207 pad 1: Net-(C208-Pad1) -> Net-(R206-Pad2)
- R207 pad 2: GND -> Net-(C209-Pad1)
- R208 pad 1: +5V -> Net-(C209-Pad1)
- R208 pad 2: Net-(Q201-C) -> GND
- R209 pad 1: Net-(Q201-C) -> Net-(C212-Pad1)
- R209 pad 2: Net-(R209-Pad2) -> GND
- R210 pad 1: Net-(R210-Pad1) -> Net-(Q201-C)
- R210 pad 2: Net-(Q201-E) -> Net-(R210-Pad2)
- R211 pad 1: Net-(Q201-E) -> +5V
- R211 pad 2: -5V -> Net-(Q201-C)
- R212 pad 1: Net-(Q201-C) -> Net-(R212-Pad1)
- R212 pad 2: Net-(Q202-B) -> Net-(Q201-E)
- R213 pad 2: Net-(Q203-B) -> -5V
- R214 pad 1: Net-(C208-Pad1) -> Net-(Q201-C)
- R214 pad 2: /MOS_G -> Net-(R210-Pad2)
- R217 pad 1: Net-(Q201-C) -> Net-(C212-Pad1)
- R217 pad 2: Net-(Q204-B) -> /MOS_G
- R218 pad 1: Net-(Q201-E) -> Net-(Q202-E)
- R218 pad 2: Net-(Q205-B) -> /MOS_G
- R221 pad 1: /MOS_G -> Net-(Q201-E)
- R221 pad 2: Net-(C210-Pad1) -> Net-(Q205-B)
- R301 pad 1: /Interface/I^{2}C_SCL -> /Interface/~{EN}
- R301 pad 2: +5V -> +3V3
- R302 pad 1: /Interface/I^{2}C_SDA -> GNDD
- R302 pad 2: +5V -> Net-(Q301-G)
- R303 pad 1: GND -> +5V
- R303 pad 2: /Interface/~{LOAD_G} -> Net-(D301-A)
- R304 pad 1: +5V -> GNDD
- R304 pad 2: Net-(D301-A) -> Net-(Q302-G)
- R305 pad 1: /Imeas -> +5V
- R305 pad 2: /Interface/Imeas+ -> Net-(D302-A)
- R306 pad 1: /OFS -> GNDD
- R306 pad 2: /Interface/Imeas- -> /Interface/CAL_MODE
- R307 pad 1: /Vmeas -> GNDD
- R307 pad 2: /Interface/Vmeas+ -> Net-(Q303-D)
- R308 pad 1: /OFS -> GNDD
- R308 pad 2: /Interface/Vmeas- -> /Interface/LOAD
- R309 pad 1: /OFS -> /Interface/SCL
- R309 pad 2: /Interface/OFSmeas -> +3V3
- R310 pad 1: GND -> GNDD
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
Commit message: aaaa
Parts:
- added R201: 0, Resistor_SMD:R_0603_1608Metric, F.Cu at (214.5, 91.8)
- R211: renamed from R210; footprint Resistor_SMD:R_0603_1608Metric -> Resistor_SMD:R_0805_2012Metric
- R215: renamed from R214; footprint Resistor_SMD:R_0603_1608Metric -> Resistor_SMD:R_0805_2012Metric
- moved J301 180.4 mm to (55.5, 68.4)
- moved J102 117.6 mm to (63.5, 69.5), turned to 180 degrees
- moved J101 98.1 mm to (79.0, 69.5), turned to 180 degrees
- moved R116 1.00 mm to (131.0, 82.7)
- renumbered R201 to R202, R202 to R203, R203 to R204, R204 to R205, R205 to R206, R206 to R207, R207 to R208, R208 to R209, R209 to R210, R211 to R212, R212 to R213, R213 to R214, R215 to R216, R216 to R217, R217 to R218, R218 to R219, R219 to R220, R220 to R221, R221 to R222, R222 to R223, R223 to R224, R224 to R225
Connections:
- C210 pad 1: +5V -> VCC
- C211 pad 1: -5V -> VEE
- FB101 pad 2: +12V -> VCC
- FB102 pad 2: -12V -> VEE
- Q202 pad 2: +5V -> VCC
- Q203 pad 3: -5V -> VEE
- Q204 pad 2: +5V -> VCC
- Q205 pad 3: -5V -> VEE
- R203 pad 1: /rt -> Net-(R201-Pad2)
- R212 pad 1: +5V -> VCC
- R214 pad 2: -5V -> VEE
- TP202 pad 1: /rt -> Net-(R201-Pad2)
- U202 pad 2: -5V -> VEE
- U202 pad 5: +5V -> VCC

Commit message: 念のため
Parts:
- removed TP203: RCTCTE, AM_Conn_TP:RCTCE
- added HS201: Heatsink_Pad_2Pin, AM_Heatsink:Heatsink_61x30x30, F.Cu at (110.2, 142.8)
- J103: value B2B-XH-A -> B2P3-VH-3.3(LF)(SN); footprint Connector_JST:JST_XH_B2B-XH-A_1x02_P2.50mm_Vertical -> Connector_JST:JST_VH_B2P3-VH_1x02_P7.92mm_Vertical
- R107, R110, R111: footprint Resistor_THT:R_Axial_DIN0207_L6.3mm_D2.5mm_P2.54mm_Vertical -> Resistor_THT:R_Axial_DIN0207_L6.3mm_D2.5mm_P10.16mm_Horizontal
- U306: footprint digikey-footprints:TO-92-3 -> Package_TO_SOT_THT:TO-92_Inline
- moved J302 212.9 mm to (54.2, 68.5)
- moved Q303 205.3 mm to (58.0, 63.0)
- moved R312 202.4 mm to (53.5, 63.0), turned to 90 degrees
- moved TP301 194.6 mm to (94.0, 12.5)
- moved RV201 190.7 mm to (73.0, 135.2)
- moved R307 190.6 mm to (60.8, 66.5), turned to -90 degrees
- moved R311 188.6 mm to (63.8, 73.2), turned to -90 degrees
- moved R214 187.2 mm to (71.0, 144.0), turned to 180 degrees
- moved U302 185.8 mm to (95.8, 33.2), turned to 90 degrees
- moved U201 185.7 mm to (72.8, 108.4), turned to 180 degrees
- moved R309 185.5 mm to (65.5, 73.2), turned to -90 degrees
- moved R301 182.2 mm to (68.2, 65.5), turned to -90 degrees
- moved U301 182.2 mm to (74.0, 66.2), turned to -90 degrees
- moved R306 181.7 mm to (70.5, 73.2), turned to 90 degrees
- moved R210 181.4 mm to (67.2, 119.4), turned to 180 degrees
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Connections:
- Q202 pad 1: Net-(Q202-E) -> Net-(Q202-B)
- Q202 pad 3: Net-(Q202-B) -> Net-(Q202-E)
- Q204 pad 1: Net-(Q204-E) -> Net-(Q204-B)
- Q204 pad 3: Net-(Q204-B) -> Net-(Q204-E)
- RV201 pad 1: Net-(R211-Pad2) -> Net-(R213-Pad1)
- RV201 pad 3: Net-(R213-Pad1) -> Net-(R211-Pad2)
- TP201 pad 1: /Imeas -> Net-(R201-Pad2)
- TP202 pad 1: Net-(R201-Pad2) -> Net-(R207-Pad2)
- U103 pad 12: /GAIN3 -> /GAIN2
- U103 pad 6: /GAIN2 -> /GAIN3
- U305 pad 1: /Interface/Imeas+ -> /Interface/Vmeas+
- U305 pad 11: /Interface/OFSmeas -> /Interface/Temp
- U305 pad 13: /Interface/Temp -> /Interface/OFSmeas
- U305 pad 2: /Interface/Imeas- -> /Interface/Vmeas-
- U305 pad 3: /Interface/Vmeas+ -> /Interface/Imeas+
- U305 pad 4: /Interface/Vmeas- -> /Interface/Imeas-
Other:
- board size 100 x 80 mm -> 100 x 100 mm
- board text added: "Bias Adjust"

Commit message: 部品配置
Parts:
- added R117: 0, Resistor_SMD:R_0805_2012Metric, F.Cu at (112.0, 80.0)
- R318, R319: moved to B.Cu
- U304: value MCP4725A0T-ECH -> MCP4726A0T-ECH
- moved P102 191.1 mm to (63.2, 145.0)
- moved R319 184.8 mm to (84.2, 77.8), turned to 90 degrees
- moved R318 175.8 mm to (97.0, 68.5), turned to 90 degrees
- moved C309 155.8 mm to (90.0, 82.2), turned to 180 degrees
- moved C306 144.8 mm to (104.2, 68.2)
- moved TP101 132.3 mm to (95.2, 89.8)
- moved C119 112.3 mm to (119.0, 114.0), turned to -90 degrees
- moved C120 110.3 mm to (124.8, 99.0), turned to 90 degrees
- moved P101 107.8 mm to (122.0, 62.5)
- moved D301 56.5 mm to (103.8, 53.0)
- moved Q301 56.5 mm to (98.2, 53.0)
- moved R302 56.5 mm to (93.8, 53.0)
- moved R303 56.5 mm to (108.8, 53.0)
- moved D302 55.8 mm to (103.8, 56.8)
- moved Q302 55.8 mm to (98.2, 56.8)
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Connections:
- R112 pad 1: Net-(U105-OUT) -> /ADC_Vref
- TP103 pad 1: Net-(U105-OUT) -> /ADC_Vref
- U105 pad 1: Net-(U105-OUT) -> /ADC_Vref
- U304 pad 6: GNDD -> /ADC_Vref
Other:
- board text added: "Load"
- board text added: "No Fault"
- board text added: "Out Fault"

Commit message: ほぼ完成?
Parts:
- added C124: 47u, Capacitor_SMD:CP_Elec_6.3x5.9, F.Cu at (144.0, 135.8)
- added C125: 47u, Capacitor_SMD:CP_Elec_6.3x5.9, F.Cu at (67.6, 132.9)
- moved C214 14.1 mm to (147.5, 122.5), turned to 180 degrees
- moved R225 7.91 mm to (145.0, 127.5), turned to 0 degrees
- moved C207 5.90 mm to (70.0, 101.8), turned to 180 degrees
- moved C208 5.63 mm to (70.0, 99.5), turned to 180 degrees
- moved R204 5.12 mm to (75.0, 101.4), turned to 180 degrees
- moved R203 5.08 mm to (75.2, 112.2)
- moved R205 5.01 mm to (75.0, 99.7), turned to 180 degrees
- moved J106 4.50 mm to (136.5, 125.2)
- moved R208 3.03 mm to (65.5, 114.2)
- moved C120 2.89 mm to (122.3, 100.5), turned to 180 degrees
- moved D101 1.50 mm to (130.8, 76.5)
- moved RLY101 1.50 mm to (140.0, 72.0)
- moved J110 1.00 mm to (141.5, 113.0)
- moved P102 0.71 mm to (63.8, 145.5)
- moved C119 0.50 mm to (119.0, 114.5)
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Connections:
- U302 pad 11: Net-(Q301-G) -> Net-(Q302-G)
- U302 pad 14: Net-(Q302-G) -> Net-(Q301-G)
- U302 pad 18: /Interface/CAL_MODE -> /Interface/LOAD
- U302 pad 19: /Interface/LOAD -> /Interface/CAL_MODE
Routing:
- net VCC: track 0.00 -> 145.2 mm, vias 0 -> 6
- net /OFS: track 0.00 -> 97.5 mm
- net Net-(Q201-C): track 0.00 -> 93.7 mm, vias 0 -> 1
- net /Imeas: track 0.00 -> 86.2 mm, vias 0 -> 3
- net VEE: track 0.00 -> 66.1 mm, vias 0 -> 4
- net /Interface/SDA: track 0.00 -> 64.2 mm, vias 0 -> 2
- net /Interface/SCL: track 0.00 -> 61.0 mm, vias 0 -> 5
- net Net-(Q201-E): track 0.00 -> 56.6 mm, vias 0 -> 1
- net /GAIN2: track 0.00 -> 54.9 mm, vias 0 -> 1
- net /GAIN0: track 0.00 -> 54.5 mm, vias 0 -> 1
- net /GAIN_SEL1: track 0.00 -> 51.2 mm
- net +3V3: track 0.00 -> 43.7 mm
- net /Interface/~{EN}: track 0.00 -> 40.5 mm, vias 0 -> 4
- net /GAIN1: track 0.00 -> 40.4 mm, vias 0 -> 1
- net /RLY_LOUT: track 0.00 -> 38.5 mm
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- added copper zone on B.Cu, net /Load+
- added copper zone on F.Cu, net /Load+
- added copper zone on B.Cu, net /MOS_D
- added copper zone on F.Cu, net /MOS_D
- added copper zone on B.Cu, net /MOS_G
- added copper zone on F.Cu, net /MOS_G
- added copper zone on B.Cu, net /MOS_S
- added copper zone on F.Cu, net /MOS_S
- added copper zone on B.Cu, net GND
- added copper zone on F.Cu, net GND
- added copper zone on In1.Cu, net GND
- added copper zone on B.Cu, net GNDA
- added copper zone on F.Cu, net GNDA
- added copper zone on B.Cu, net GNDD
- added copper zone on F.Cu, net GNDD
- added copper zone on In1.Cu, net GNDD

Commit message: ほぼ完成
Parts:
- FB101, FB102: footprint Inductor_SMD:L_0805_2012Metric -> Inductor_THT:L_Axial_L5.3mm_D2.2mm_P2.54mm_Vertical_Vishay_IM-1
- moved FB102 1.90 mm to (64.5, 126.1)
- moved FB101 1.70 mm to (64.5, 139.9)
Connections:
- U104 pad 3: /Vin -> GNDA
- U104 pad 5: GNDA -> /Vin
Routing:
- net +3V3: track 43.7 -> 338.6 mm, vias 0 -> 21
- net +5V: track 29.4 -> 147.2 mm, vias 2 -> 5
- net -3V3: track 18.0 -> 128.8 mm, vias 0 -> 6
- net GNDA: track 14.6 -> 121.2 mm, vias 0 -> 3
- net /Interface/Vmeas+: track 6.10 -> 25.0 mm, vias 0 -> 2
- net /Interface/Imeas+: track 6.70 -> 25.0 mm, vias 0 -> 2
- net /Interface/Temp: track 17.4 -> 30.9 mm, vias 0 -> 2
- net VEE: track 66.1 -> 76.9 mm, vias 4 -> 5
- net /Vin: track 18.1 -> 27.8 mm, vias 0 -> 1
- net Net-(Q205-E): track 0.00 -> 5.53 mm
- net Net-(Q203-E): track 0.00 -> 5.51 mm
- net Net-(Q204-E): track 0.00 -> 5.51 mm
- net Net-(Q202-E): track 0.00 -> 5.49 mm
- net Net-(C214-Pad1): track 0.00 -> 5.19 mm
- net Net-(R107-Pad2): track 6.60 -> 11.5 mm, vias 0 -> 2
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- added copper zone on B.Cu, net +3V3
- added copper zone on In2.Cu, net GNDA

Commit message: アノテーション変更前
Parts:
- added J111: B2B-XH-A, Connector_JST:JST_XH_B2B-XH-A_1x02_P2.50mm_Vertical, F.Cu at (56.5, 116.0)
- added J112: PH-1X3SG, Connector_PinHeader_2.54mm:PinHeader_1x03_P2.54mm_Vertical, F.Cu at (84.5, 118.0)
- moved C103 8.51 mm to (63.5, 108.0), turned to 90 degrees
- moved C209 5.21 mm to (68.2, 115.5), turned to 90 degrees
- moved TP202 2.37 mm to (63.0, 120.0)
- moved R207 1.68 mm to (65.0, 111.0), turned to -90 degrees
- moved R208 1.46 mm to (64.8, 115.5), turned to -90 degrees
- moved C211 1.35 mm to (67.2, 119.0)
- moved R210 1.35 mm to (67.2, 120.8)
- moved R201 1.25 mm to (80.8, 113.2)
- moved R209 0.85 mm to (66.5, 115.5), turned to 90 degrees
Connections:
- U304 pad 1: /rt -> /Interface/rt
Routing:
- net /Interface/rt: track 0.00 -> 41.8 mm, vias 0 -> 2
- net /rt: track 38.4 -> 4.54 mm, vias 2 -> 0
- net Net-(J111-Pin_1): track 0.00 -> 24.6 mm
- net GND: track 1.62 -> 13.5 mm, vias 16 -> 15
- net Net-(C207-Pad1): track 0.00 -> 8.96 mm
- net +3V3: track 338.6 -> 344.7 mm
- net Net-(C205-Pad2): track 21.2 -> 23.2 mm
- net Net-(C209-Pad1): track 5.02 -> 7.06 mm
- net Net-(R207-Pad2): track 10.4 -> 9.00 mm
- net Net-(J102-Pin_1): track 23.9 -> 22.9 mm
- net VCC: track 142.8 -> 141.8 mm
- net Net-(R201-Pad2): track 10.6 -> 9.90 mm
- net Net-(C212-Pad1): track 10.1 -> 10.6 mm
- net VEE: track 76.9 -> 77.4 mm
- net /Imeas: vias 2 -> 3
