File: PI.kicad_sch (KiCad schematic)
At the start: 45 parts, among them Q3 2SC1815, Q4 MTBT3906, Q5 MTBT3904, Q6 2SD1415A, Q7 TTB1020B, Q8 2SD1415A, Q9 TTB1020B, U12 KIA75S358F, U4 ADA4522-1ARZ

Commit message: aaaa
Parts:
- removed C2: 0.01u(FL), Capacitor_THT:C_Rect_L7.0mm_W2.5mm_P5.00mm, symbol Device:C_Small
- removed C29: 100p, Capacitor_SMD:C_0603_1608Metric, symbol Device:C_Small
- removed Q4: MTBT3906, Package_TO_SOT_THT:TO-92S, symbol Transistor_BJT:Q_PNP_BEC
- removed Q5: MTBT3904, symbol Transistor_BJT:Q_NPN_ECB
- removed R10: 0, Resistor_THT:R_Axial_DIN0207_L6.3mm_D2.5mm_P2.54mm_Vertical, symbol Device:R
- removed R29, R33: 10k, symbol Device:R
- removed R32: 100k, symbol Device:R
- removed R37: 300, symbol Device:R
- removed RV5, RV6: 50k, symbol Device:R_Potentiometer_Trim
- added C203: 0.01u(FL), Capacitor_SMD:C_0805_2012Metric, symbol Device:C_Small
- added C205: NC, Capacitor_SMD:C_0805_2012Metric, symbol Device:C_Small
- added C210: 1000p, Capacitor_SMD:C_0805_2012Metric, symbol Device:C_Small
- added C211: 10p, Capacitor_SMD:C_0603_1608Metric, symbol Device:C_Small
- added C212: 0.047u(FL), Capacitor_THT:C_Rect_L7.2mm_W5.0mm_P5.00mm, symbol Device:C_Small
- added R203, R205: 0, Resistor_SMD:R_0603_1608Metric, symbol Device:R
- added R204, R216: 1k, Resistor_SMD:R_0603_1608Metric, symbol Device:R
- added R213: 33k, Resistor_SMD:R_0603_1608Metric, symbol Device:R
- added R223: 4.7, Resistor_SMD:R_2512_6332Metric, symbol Device:R
- added TP203: RCTCTE, symbol Connector:TestPoint_Probe
- C201: renamed from C22; Akizuki_code (none) -> 105728
- C202: renamed from C23; Akizuki_code (none) -> 105728
- C204: renamed from C10; value 0.1u -> NC
- C206: renamed from C3; footprint Capacitor_THT:C_Rect_L7.0mm_W2.5mm_P5.00mm -> Capacitor_SMD:C_0805_2012Metric; Akizuki_code 116112 -> 115631
- C207: renamed from C27; Akizuki_code (none) -> 105728
- C208: renamed from C11; value 0.1u -> NC
- C209: renamed from C28; Akizuki_code (none) -> 105728
- Q201: renamed from Q3; footprint (none) -> Package_TO_SOT_THT:TO-92L_Inline; Akizuki_code (none) -> 117089
- Q202: renamed from Q6; footprint (none) -> Package_TO_SOT_THT:TO-220-3_Vertical; Akizuki_code (none) -> 110058; Akizuki_code2 (none) -> 106369
- Q203: renamed from Q7; footprint Package_TO_SOT_THT:TO-92S -> Package_TO_SOT_THT:TO-220-3_Vertical; Akizuki_code (none) -> 117309
- Q204: renamed from Q8; footprint (none) -> Package_TO_SOT_THT:TO-220-3_Vertical; Akizuki_code (none) -> 110058; Akizuki_code2 (none) -> 106369
- Q205: renamed from Q9; footprint Package_TO_SOT_THT:TO-92S -> Package_TO_SOT_THT:TO-220-3_Vertical; Akizuki_code (none) -> 117309
- R201: renamed from R12; footprint Resistor_THT:R_Axial_DIN0207_L6.3mm_D2.5mm_P2.54mm_Vertical -> Resistor_SMD:R_0603_1608Metric; Akizuki_code (none) -> 106668
- R202: renamed from R28; footprint Resistor_THT:R_Axial_DIN0207_L6.3mm_D2.5mm_P2.54mm_Vertical -> Resistor_SMD:R_0603_1608Metric
- R206: renamed from R46; footprint Resistor_THT:R_Axial_DIN0207_L6.3mm_D2.5mm_P2.54mm_Vertical -> Resistor_SMD:R_0603_1608Metric
- R207: renamed from R11; footprint Resistor_THT:R_Bare_Metal_Element_L16.3mm_W4.8mm_P15.30mm -> Resistor_SMD:R_0603_1608Metric
- R208: renamed from R31; value 10k -> 100k; footprint Resistor_THT:R_Bare_Metal_Element_L16.3mm_W4.8mm_P15.30mm -> Resistor_SMD:R_0603_1608Metric
- R209: renamed from R34; value 10k -> 3.3k; footprint (none) -> Resistor_SMD:R_0603_1608Metric
- R210: renamed from R30; value 20k -> 510; footprint (none) -> Resistor_SMD:R_2512_6332Metric; Sengoku_code (none) -> EEHD-0ECM
- R211: renamed from R35; value 10k -> 1k; footprint (none) -> Resistor_SMD:R_0805_2012Metric; Sengoku_code (none) -> EEHD-57BZ
- R212: renamed from R36; value 20k -> 510; footprint (none) -> Resistor_SMD:R_2512_6332Metric; Sengoku_code (none) -> EEHD-0ECM
- R214: renamed from R40; footprint (none) -> Resistor_SMD:R_1206_3216Metric; Sengoku_code (none) -> EEHD-57BS
- R215: renamed from R41; footprint (none) -> Resistor_SMD:R_1206_3216Metric; Sengoku_code (none) -> EEHD-57BS
- R219: renamed from R42; footprint (none) -> Resistor_SMD:R_1206_3216Metric; Sengoku_code (none) -> EEHD-57BS
- R220: renamed from R43; footprint (none) -> Resistor_SMD:R_1206_3216Metric; Sengoku_code (none) -> EEHD-57BS
- RV201: renamed from RV7; value 10k -> 2k; footprint (none) -> AM_Potentiometer:TSR-065-xxx-R
- TP201: renamed from TP4; value FeedBack -> RCTCTE; footprint TestPoint:TestPoint_Loop_D2.50mm_Drill1.0mm -> (none)
- TP202: renamed from TP5; value Set -> RCTCTE; footprint TestPoint:TestPoint_Loop_D2.50mm_Drill1.0mm -> (none)
- U201: renamed from U4; footprint Package_DIP:DIP-8_W7.62mm -> Package_SO:SOIC-8_3.9x4.9mm_P1.27mm; AkizukiCode 114063 -> (none); Akizuki_code2 (none) -> 114063
- renumbered R38 to R217, R39 to R218, R44 to R221, R45 to R222, U12 to U202
Connections:
- net GNDA is gone; now on net GND: C204.2, C208.2, R207.2, R208.2
- net GND: now also C212.2
- net ut_buf: now also C211.2, R216.2, R223.1
- net yt: now also C203.1
- net at C206.2, U201.6: now also C205.2, R204.2, R205.1; no longer R206.1
- net at R214.1, R219.1: now also Q201.2 (C), R209.1, R210.2, U202.4, C210.2, R213.1
- net at R215.1, R220.1: now also Q201.1 (E), R211.2, R212.1
- net at R208.1, U202.3: now also C210.1, C211.1, R216.1
- net at R201.2, U201.2: now also C203.2, C205.1, R203.1, R204.1
- net at R209.2, RV201.1: now also R213.2
- net at C206.1: now also R203.2
- net at R211.1, RV201.3: no longer Q201.3 (B), RV201.2
- net +12V renamed +5V
- net -12V renamed -5V
- new net: R205.2, R206.1, TP203.1
- new net: C212.1, R223.2
- new net: Q201.3 (B), RV201.2
Other:
- note added: "・C208, C209, R221, C210は発振止めのオプション 適宜つける"
- note added: "・DCゲインあげすぎると多分発振する"
- note added: "負荷素子: BJT ・+5Vは2A位の容量はとれるようにする ・-5Vは動作しないので適当な容量 負荷素子: MOOSFET, IGBT ・±5V→±12Vに変更 ・適当にバイアスの抵抗も変える ・電源は2,300mA程度?"
- moved on the sheet: C201, C202, C204, C206, C207, C208, C209, Q201, Q202, Q203, Q204, Q205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

Commit message: kannsei
Parts:
- removed C207, C209: 0.1u, Capacitor_SMD:C_0603_1608Metric, symbol Device:C_Small
- added C205: NC, Capacitor_SMD:C_0805_2012Metric, symbol Device:C_Small
- added C208: 1000p(FL), Capacitor_SMD:C_0805_2012Metric, symbol Device:C_Small
- added C210, C211: 0.1u, Capacitor_SMD:C_0603_1608Metric, symbol Device:C_Small
- added R201: 0, Resistor_SMD:R_0603_1608Metric, symbol Device:R
- added R205: 1M, Resistor_SMD:R_0603_1608Metric, symbol Device:R
- C207: renamed from C206; value 0.01u(FL) -> 1000p(FL)
- R202: renamed from R201; value 10k -> 1k
- R204: renamed from R203; value 0 -> 1M
- R206: renamed from R204; value 1k -> NC; now not fitted
- R211: renamed from R209; footprint Resistor_SMD:R_0603_1608Metric -> Resistor_SMD:R_0805_2012Metric
- R215: renamed from R213; footprint Resistor_SMD:R_0603_1608Metric -> Resistor_SMD:R_0805_2012Metric
- R219: renamed from R217; value 0.1 -> 1; footprint (none) -> Resistor_THT:R_Box_L14.0mm_W5.0mm_P9.00mm
- R220: renamed from R218; value 0.1 -> 1; footprint (none) -> Resistor_THT:R_Box_L14.0mm_W5.0mm_P9.00mm
- R223: renamed from R221; value 0.1 -> 1; footprint (none) -> Resistor_THT:R_Box_L14.0mm_W5.0mm_P9.00mm
- R224: renamed from R222; value 0.1 -> 1; footprint (none) -> Resistor_THT:R_Box_L14.0mm_W5.0mm_P9.00mm
- TP201, TP202, TP203: footprint (none) -> AM_Conn_TP:RCTCE
- renumbered C205 to C206, C208 to C209, C210 to C212, C211 to C213, C212 to C214, R202 to R203, R205 to R207, R206 to R208, R207 to R209, R208 to R210, R210 to R212, R211 to R213, R212 to R214, R214 to R216, R215 to R217, R216 to R218, R219 to R221, R220 to R222, R223 to R225
Connections:
- net +5V is gone; now on net VCC: Q202.2 (C), Q204.2 (C), R212.1, U202.5 (VCC)
- net -5V is gone; now on net VEE: Q203.3 (C), Q205.3 (C), R214.2, U202.2 (VEE)
- net +3V3: now also C201.1
- net -3V3: now also C202.1
- net GND: now also C210.2, C211.2
- net VCC: now also C210.1; no longer C201.1
- net VEE: now also C211.1; no longer C202.1
- net rt: now also R201.1; no longer R203.1, TP202.1
- net at C206.2, C207.2, R206.2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: now also C205.2, C208.2
- net at C203.2, C206.1, R202.2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: now also C205.1, R205.1
- net at C207.1, R204.2: now also C208.1, R205.2
- new net: R201.2, R203.1, TP202.1
Other:
- note removed: "・C208, C209, R221, C210は発振止めのオプション 適宜つける"
- note removed: "・DCゲインあげすぎると多分発振する"
- note removed: "負荷素子: BJT ・+5Vは2A位の容量はとれるようにする ・-5Vは動作しないので適当な容量 負荷素子: MOOSFET, IGBT ・±5V→±12Vに変更 ・適当にバイアスの抵抗も変える ・電源は2,300mA程度?"
- company: (none) -> EosinY
- title: (none) -> Analog Controller
- moved on the sheet: C206, C207, R204, TP202, U201

Commit message: 念のため
Parts:
- removed TP201: RCTCTE, AM_Conn_TP:RCTCE, symbol Connector:TestPoint_Probe
- added HS201: Heatsink_Pad_2Pin, AM_Heatsink:Heatsink_61x30x30, symbol Mechanical:Heatsink_Pad_2Pin
- Q202, Q204: symbol Transistor_BJT:Q_NPN_ECB -> Transistor_BJT:Q_NPN_BCE
- renumbered TP202 to TP201, TP203 to TP202
Connections:
- net at R211.2, R215.2: now also RV201.3; no longer RV201.1
- net at Q202.1 (B): now also R216.2; no longer R219.1
- net at Q202.3 (E): now also R219.1; no longer R216.2
- net at R213.1: now also RV201.1; no longer RV201.3
- net at R221.2: now also Q204.1 (B); no longer Q204.3 (B)
- net at R223.1: now also Q204.3 (E); no longer Q204.1 (E)
- no-connect marks 0 -> 2
Changed lines of the file:
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@@
 		(color 0 0 0 0)
 	)
+	(no_connect
+		(at 259.08 90.17)
+	)
+	(no_connect
+		(at 254 90.17)
+	)
 	(wire
 		(pts
@@
 	)
 	(symbol
-		(lib_id "Transistor_BJT:Q_NPN_ECB")
+		(lib_id "Transistor_BJT:Q_NPN_BCE")
 		(at 193.04 83.82 0)
 		(unit 1)
@@
 			)
 		)
-		(property "Description" "NPN transistor, emitter/collector/base"
+		(property "Description" "NPN transistor, base/collector/emitter"
 			(at 193.04 83.82 0)
 			(hide yes)
@@
 			)
 		)
-		(property "Sim.Pins" "1=E 2=C 3=B"
+		(property "Sim.Pins" "1=B 2=C 3=E"
 			(at 193.04 83.82 0)
 			(hide yes)
@@
 	)
 	(symbol
+		(lib_id "Mechanical:Heatsink_Pad_2Pin")
+		(at 256.54 87.63 0)
+		(unit 1)
+		(body_style 1)
+		(exclude_from_sim no)
+		(in_bom yes)
+		(on_board yes)
+		(in_pos_files yes)
+		(dnp no)
+		(fields_autoplaced yes)
+		(property "Reference" "HS201"
+			(at 260.35 85.7249 0)
+			(show_name no)
+			(do_not_autoplace no)
+			(effects
+				(font
+					(size 1.27 1.27)
+				)
+				(justify left)
+			)
+		)
+		(property "Value" "Heatsink_Pad_2Pin"
+			(at 260.35 88.2649 0)
+			(show_name no)
+			(do_not_autoplace no)
+			(effects
+				(font
+					(size 1.27 1.27)
+				)
+				(justify left)
+			)
+		)
+		(property "Footprint" "AM_Heatsink:Heatsink_61x30x30"
+			(at 256.8448 88.9 0)
+			(hide yes)
+			(show_name no)
+			(do_not_autoplace no)
+			(effects
+				(font
+					(size 1.27 1.27)
+				)
+			)
+		)
+		(property "Datasheet" ""
+			(at 256.8448 88.9 0)
+			(hide yes)
+			(show_name no)
+			(do_not_autoplace no)
+			(effects
+				(font
+					(size 1.27 1.27)
+				)
+			)
+		)
+		(property "Description" "Heatsink with electrical connection, 2 pin"
+			(at 256.54 87.63 0)
+			(hide yes)
+			(show_name no)
+			(do_not_autoplace no)
+			(effects
+				(font
+					(size 1.27 1.27)
+				)
+			)
+		)
+		(pin "2"
+		)
+		(pin "1"
+		)
+		(instances
+			(project "Main_SMD_Controller_v2"
+				(path "/ad678d38-2bf7-47ec-94cd-212edb6f07b2/4cb88ddc-3883-4645-847c-692dc35751fd"
+					(reference "HS201")
+					(unit 1)
+				)
+			)
+		)
+	)
+	(symbol
 		(lib_id "power:-3V3")
 		(at 66.04 95.25 180)
@@
 	)
 	(symbol
-		(lib_id "Transistor_BJT:Q_NPN_ECB")
+		(lib_id "Transistor_BJT:Q_NPN_BCE")
 		(at 227.33 83.82 0)
 		(unit 1)
@@
 			)
 		)
-		(property "Description" "NPN transistor, emitter/collector/base"
+		(property "Description" "NPN transistor, base/collector/emitter"
 			(at 227.33 83.82 0)
 			(hide yes)
@@
 			)
 		)
-		(property "Sim.Pins" "1=E 2=C 3=B"
+		(property "Sim.Pins" "1=B 2=C 3=E"
 			(at 227.33 83.82 0)
 			(hide yes)
@@
 	)
 	(symbol
-		(lib_id "Connector:TestPoint_Probe")
-		(at 36.83 85.09 0)
-		(mirror y)
-		(unit 1)
-		(body_style 1)
-		(exclude_from_sim no)
-		(in_bom yes)
-		(on_board yes)
-		(in_pos_files yes)
-		(dnp no)
-		(property "Reference" "TP201"
-			(at 33.02 82.2324 0)
-			(show_name no)
-			(do_not_autoplace no)
-			(effects
-				(font
-					(size 1.27 1.27)
-				)
-				(justify left)
-			)
-		)
-		(property "Value" "RCTCTE"
-			(at 33.02 84.7724 0)
-			(show_name no)
-			(do_not_autoplace no)
-			(effects
-				(font
-					(size 1.27 1.27)
-				)
-				(justify left)
-			)
-		)
-		(property "Footprint" "AM_Conn_TP:RCTCE"
-			(at 31.75 85.09 0)
-			(hide yes)
-			(show_name no)
-			(do_not_autoplace no)
-			(effects
-				(font
-					(size 1.27 1.27)
-				)
-			)
-		)
-		(property "Datasheet" ""
-			(at 31.75 85.09 0)
-			(hide yes)
-			(show_name no)
-			(do_not_autoplace no)
-			(effects
-				(font
-					(size 1.27 1.27)
-				)
-			)
-		)
-		(property "Description" "test point (alternative probe-style design)"
-			(at 36.83 85.09 0)
-			(hide yes)
-			(show_name no)
-			(do_not_autoplace no)
-			(effects
-				(font
-					(size 1.27 1.27)
-				)
-			)
-		)
-		(property "Description_1" ""
-			(at 36.83 85.09 0)
-			(hide yes)
-			(show_name no)
-			(do_not_autoplace no)
-			(effects
-				(font
-					(size 1.27 1.27)
-				)
-			)
-		)
-		(property "Sengoku_code" ""
-			(at 36.83 85.09 0)
-			(hide yes)
-			(show_name no)
-			(do_not_autoplace no)
-			(effects
-				(font
-					(size 1.27 1.27)
-				)
-			)
-		)
-		(pin "1"
-		)
-		(instances
-			(project "Main_SMD_Controller_v2"
-				(path "/ad678d38-2bf7-47ec-94cd-212edb6f07b2/4cb88ddc-3883-4645-847c-692dc35751fd"
-					(reference "TP201")
-					(unit 1)
-				)
-			)
-		)
-	)
-	(symbol
 		(lib_id "Device:R")
 		(at 195.58 95.25 0)
@@
 		(lib_id "Device:R_Potentiometer_Trim")
 		(at 156.21 104.14 0)
+		(mirror x)
 		(unit 1)
 		(body_style 1)
@@
 		(dnp no)
 		(property "Reference" "RV201"
-			(at 153.67 102.8699 0)
+			(at 153.67 105.4101 0)
 			(show_name no)
 			(do_not_autoplace no)
@@
 		)
 		(property "Value" "2k"
-			(at 153.67 105.4099 0)
+			(at 153.67 102.8701 0)
 			(show_name no)
 			(do_not_autoplace no)
@@
 		(in_pos_files yes)
 		(dnp no)
-		(property "Reference" "TP203"
+		(property "Reference" "TP202"
 			(at 98.298 83.566 0)
 			(show_name no)
@@
 			(project "Main_SMD_Controller_v2"
 				(path "/ad678d38-2bf7-47ec-94cd-212edb6f07b2/4cb88ddc-3883-4645-847c-692dc35751fd"
-					(reference "TP203")
+					(reference "TP202")
 					(unit 1)
 				)
@@
 		(in_pos_files yes)
 		(dnp no)
-		(property "Reference" "TP202"
+		(property "Reference" "TP201"
 			(at 35.56 102.87 0)
 			(show_name no)
@@
 			(project "Main_SMD_Controller_v2"
 				(path "/ad678d38-2bf7-47ec-94cd-212edb6f07b2/4cb88ddc-3883-4645-847c-692dc35751fd"
-					(reference "TP202")
+					(reference "TP201")
 					(unit 1)
 				)

Commit message: できたかも
Parts:
- C201, C202, C210, C211: Akizuki_code2 (none) -> 116143
- C207: Sengoku_code (none) -> EEHD-5PLN
- C212: value 1000p -> 1000p(FL); Akizuki_code 115632 -> 115631
- HS201: Akizuki_code (none) -> 112537
- R201, R203, R207, R208: Akizuki_code (none) -> 111619
- R202: Akizuki_code 106668 -> 114122
- R204, R205: Akizuki_code 10668 -> 130359
- R209: Akizuki_code 106668 -> 115029
- R210: Akizuki_code 106668 -> 115321
- R211: Sengoku_code (none) -> EEHD-57C5
- R215: Sengoku_code (none) -> EEHD-57CH
- R218: Akizuki_code 10668 -> 114122
- R219, R220, R223, R224: Akizuki_code (none) -> 110701
- RV201: Akizuki_code (none) -> 106061
- TP201, TP202: Akizuki_code (none) -> 131773
- U201: Akizuki_code (none) -> 115092
- U202: Akizuki_code (none) -> 109229

Commit message: 現状確定
Parts:
- C201, C202, C210, C211: In_Stock (none) -> 77
- C207, C212, R211, R212, R213, R214, R215, R216, R217, R219, R220, R221, R222, R223, R224, TP201, TP202, U202: In_Stock (none) -> 0
- C208: In_Stock (none) -> 0; Sengoku_code (none) -> EEHD-5PLN; now fitted
- HS201, Q203, Q205: In_Stock (none) -> 1
- Q201: In_Stock (none) -> 61
- Q202, Q204: In_Stock (none) -> 4
- R201, R203, R207, R208: In_Stock (none) -> 92
- R202, R218: In_Stock (none) -> 170
- R204, R205: In_Stock (none) -> 75
- R209: In_Stock (none) -> >100
- R210: In_Stock (none) -> 50
- RV201: In_Stock (none) -> 21
- U201: In_Stock (none) -> 2
Other:
- moved on the sheet: C201, C202, C203, C204, C205, C206, C207, C209, C210, C211, C212, C213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
